File: hw/PIB/monarch_payload_interface_board_rev1/_autosave-monarch_payload_interface_board_rev1.kicad_pcb (KiCad board)
At the start: 2 copper layers, 96 x 89.9 mm, 7 parts, among them U1 Payload, U2 STM32L4A6VGTx, U3 NZT7053

Commit message: Components selection for valves so far
Parts:
- removed the D1 at (133.2, 71.9)
- moved R1 26.2 mm to (112.1, 65.7)
- moved D1 24.6 mm to (118.0, 59.5), turned to 90 degrees
- moved CR1 8.07 mm to (114.5, 59.3), turned to 90 degrees

Commit message: More components
Parts:
- removed D1: 1SMA4757, Zener_diode:DIOM4325X250N
- removed U3: NZT7053, nzt7:SOT-223_ONS-L
- added C1: 100nF, Capacitor_SMD:C_0603_1608Metric, F.Cu at (173.0, 79.5)
- added C10: 22u, Capacitor_SMD:C_0603_1608Metric, F.Cu at (173.0, 99.5)
- added C11: 100n, Capacitor_SMD:C_0603_1608Metric, F.Cu at (175.9, 104.1)
- added C12: 100n, Capacitor_SMD:C_0603_1608Metric, F.Cu at (175.9, 106.6)
- added C13: 100n, Capacitor_SMD:C_0603_1608Metric, F.Cu at (175.9, 109.1)
- added C14: 100n, Capacitor_SMD:C_0603_1608Metric, F.Cu at (175.9, 111.6)
- added C15: 100n, Capacitor_SMD:C_0603_1608Metric, F.Cu at (175.9, 114.1)
- added C16: 4.7u, Capacitor_SMD:C_0603_1608Metric, F.Cu at (179.9, 104.1)
- added C17: 100n, Capacitor_SMD:C_0603_1608Metric, F.Cu at (179.9, 106.6)
- added C18: 1u, Capacitor_SMD:C_0603_1608Metric, F.Cu at (179.9, 109.1)
- added C19: 10n, Capacitor_SMD:C_0603_1608Metric, F.Cu at (179.9, 111.6)
- added C2: 82uF, 35SVT82M:CAP_35SVT82M, F.Cu at (148.9, 55.9)
- added C20: 1u, Capacitor_SMD:C_0603_1608Metric, F.Cu at (179.9, 114.1)
- added C3: 10uF, Capacitor_SMD:C_0603_1608Metric, F.Cu at (173.0, 82.0)
- added C4: 8.2n, Capacitor_SMD:C_0603_1608Metric, F.Cu at (173.0, 84.5)
- added C5: 22p, Capacitor_SMD:C_0603_1608Metric, F.Cu at (173.0, 87.0)
- added C6: 3.3p, Capacitor_SMD:C_0603_1608Metric, F.Cu at (173.0, 89.5)
- added C7: 2.2u, Capacitor_SMD:C_0603_1608Metric, F.Cu at (173.0, 92.0)
- added C8: 100n, Capacitor_SMD:C_0603_1608Metric, F.Cu at (173.0, 94.5)
- added C9: 22u, Capacitor_SMD:C_0603_1608Metric, F.Cu at (173.0, 97.0)
- added CR10: S1J-13-F, s1j:SMA_DIO-L, F.Cu at (128.3, 66.1)
- added CR11: S1J-13-F, s1j:SMA_DIO-L, F.Cu at (128.3, 70.4)
- added CR12: S1J-13-F, s1j:SMA_DIO-L, F.Cu at (128.3, 74.7)
- added CR13: S1J-13-F, s1j:SMA_DIO-L, F.Cu at (137.0, 53.1)
- added CR14: S1J-13-F, s1j:SMA_DIO-L, F.Cu at (137.0, 57.4)
- added CR15: S1J-13-F, s1j:SMA_DIO-L, F.Cu at (137.0, 61.7)
- added CR16: S1J-13-F, s1j:SMA_DIO-L, F.Cu at (137.0, 66.1)
- added CR17: S1J-13-F, s1j:SMA_DIO-L, F.Cu at (137.0, 70.4)
- added CR18: S1J-13-F, s1j:SMA_DIO-L, F.Cu at (137.0, 74.7)
- added CR2: S1J-13-F, s1j:SMA_DIO-L, F.Cu at (119.6, 57.4)
- added CR3: S1J-13-F, s1j:SMA_DIO-L, F.Cu at (119.6, 61.7)
- added CR4: S1J-13-F, s1j:SMA_DIO-L, F.Cu at (119.6, 66.1)
- added CR5: S1J-13-F, s1j:SMA_DIO-L, F.Cu at (119.6, 70.4)
- added CR6: S1J-13-F, s1j:SMA_DIO-L, F.Cu at (119.6, 74.7)
- added CR7: S1J-13-F, s1j:SMA_DIO-L, F.Cu at (128.3, 53.1)
- added CR8: S1J-13-F, s1j:SMA_DIO-L, F.Cu at (128.3, 57.4)
- added CR9: S1J-13-F, s1j:SMA_DIO-L, F.Cu at (128.3, 61.7)
- added L1: XEL4020-561MEC, XEL:IND_XEL4020_COC-L, F.Cu at (146.1, 63.6)
- added Q1: FZT600TA, fzt:SOT230P700X170-4N, F.Cu at (109.7, 55.0)
- added Q10: FZT600TA, fzt:SOT230P700X170-4N, F.Cu at (145.8, 82.3)
- added Q11: FZT600TA, fzt:SOT230P700X170-4N, F.Cu at (145.8, 90.6)
- added Q12: FZT600TA, fzt:SOT230P700X170-4N, F.Cu at (145.8, 98.8)
- added Q13: FZT600TA, fzt:SOT230P700X170-4N, F.Cu at (145.8, 107.1)
- added Q14: FZT600TA, fzt:SOT230P700X170-4N, F.Cu at (145.8, 115.3)
- added Q15: FZT600TA, fzt:SOT230P700X170-4N, F.Cu at (155.4, 82.3)
- added Q16: FZT600TA, fzt:SOT230P700X170-4N, F.Cu at (155.4, 90.6)
- added Q17: FZT600TA, fzt:SOT230P700X170-4N, F.Cu at (155.4, 98.8)
- added Q18: FZT600TA, fzt:SOT230P700X170-4N, F.Cu at (155.4, 107.1)
- added Q2: FZT600TA, fzt:SOT230P700X170-4N, F.Cu at (109.7, 63.3)
- added Q3: FZT600TA, fzt:SOT230P700X170-4N, F.Cu at (109.7, 71.5)
- added Q4: FZT600TA, fzt:SOT230P700X170-4N, F.Cu at (109.7, 79.8)
- added Q5: FZT600TA, fzt:SOT230P700X170-4N, F.Cu at (136.2, 82.3)
- added Q6: FZT600TA, fzt:SOT230P700X170-4N, F.Cu at (136.2, 90.6)
- added Q7: FZT600TA, fzt:SOT230P700X170-4N, F.Cu at (136.2, 98.8)
- added Q8: FZT600TA, fzt:SOT230P700X170-4N, F.Cu at (136.2, 107.1)
- added Q9: FZT600TA, fzt:SOT230P700X170-4N, F.Cu at (136.2, 115.3)
- added R10: 125, Resistor_SMD:R_0402_1005Metric, F.Cu at (164.6, 83.2)
- added R11: 125, Resistor_SMD:R_0402_1005Metric, F.Cu at (164.6, 85.2)
- added R12: 125, Resistor_SMD:R_0402_1005Metric, F.Cu at (164.6, 87.2)
- added R13: 125, Resistor_SMD:R_0402_1005Metric, F.Cu at (164.6, 89.2)
- added R14: 125, Resistor_SMD:R_0402_1005Metric, F.Cu at (164.6, 91.2)
- added R15: 125, Resistor_SMD:R_0402_1005Metric, F.Cu at (167.5, 79.2)
- added R16: 125, Resistor_SMD:R_0402_1005Metric, F.Cu at (167.5, 81.2)
- added R17: 187k, Resistor_SMD:R_0402_1005Metric, F.Cu at (176.4, 79.2)
- added R18: 825k, Resistor_SMD:R_0402_1005Metric, F.Cu at (176.4, 81.2)
- added R19: 92k, Resistor_SMD:R_0402_1005Metric, F.Cu at (176.4, 83.2)
- added R2: 125, Resistor_SMD:R_0402_1005Metric, F.Cu at (161.7, 81.2)
- added R20: 51.1k, Resistor_SMD:R_0402_1005Metric, F.Cu at (176.4, 85.2)
- added R21: 205k, Resistor_SMD:R_0402_1005Metric, F.Cu at (176.4, 87.2)
- added R22: 4.7k, Resistor_SMD:R_0402_1005Metric, F.Cu at (172.4, 103.8)
- added R23: 4.7k, Resistor_SMD:R_0402_1005Metric, F.Cu at (172.4, 105.8)
- added R24: 4.7k, Resistor_SMD:R_0402_1005Metric, F.Cu at (172.4, 107.8)
- added R25: 4.7k, Resistor_SMD:R_0402_1005Metric, F.Cu at (172.4, 109.8)
- added R26: 4.7k, Resistor_SMD:R_0402_1005Metric, F.Cu at (172.4, 111.8)
- added R27: 4.7k, Resistor_SMD:R_0402_1005Metric, F.Cu at (172.4, 113.8)
- added R28: 4.7k, Resistor_SMD:R_0402_1005Metric, F.Cu at (172.4, 115.7)
- added R29: 4.7k, Resistor_SMD:R_0402_1005Metric, F.Cu at (172.4, 117.7)
- added R3: 125, Resistor_SMD:R_0402_1005Metric, F.Cu at (161.7, 83.2)
- added R30: 125, Resistor_SMD:R_0402_1005Metric, F.Cu at (167.5, 83.2)
- added R31: 125, Resistor_SMD:R_0402_1005Metric, F.Cu at (167.5, 85.2)
- added R4: 125, Resistor_SMD:R_0402_1005Metric, F.Cu at (161.7, 85.2)
- added R5: 125, Resistor_SMD:R_0402_1005Metric, F.Cu at (161.7, 87.2)
- added R6: 125, Resistor_SMD:R_0402_1005Metric, F.Cu at (161.7, 89.2)
- added R7: 125, Resistor_SMD:R_0402_1005Metric, F.Cu at (161.7, 91.2)
- added R8: 125, Resistor_SMD:R_0402_1005Metric, F.Cu at (164.6, 79.2)
- added R9: 125, Resistor_SMD:R_0402_1005Metric, F.Cu at (164.6, 81.2)
- added U4: TPS61088QRHLRQ1, tps6:RHL0020A, F.Cu at (177.5, 91.2)
- R1: value RMCF1206JT330R -> 125; footprint 330O res:STA_RMCF1206_STP -> Resistor_SMD:R_0402_1005Metric
- moved R1 51.4 mm to (161.7, 79.2)
- moved CR1 8.07 mm to (119.6, 53.1), turned to 0 degrees
- moved U2 4.93 mm to (117.2, 93.0), turned to 180 degrees
Connections:
- CR1 pad 1: unconnected-(CR1-Pad1) -> /PC104_stack/12VA
- CR1 pad 2: unconnected-(CR1-Pad2) -> /Valves/Valve1-
- R1 pad 1: unconnected-(R1-Pad1) -> /MCU/Valve1
- R1 pad 2: unconnected-(R1-Pad2) -> Net-(Q1-B)
- U1 pad 100: unconnected-(U1-48-Pad100) -> GND
- U1 pad 33: unconnected-(U1-Pad33) -> /MCU/UART_TX
- U1 pad 35: unconnected-(U1-Pad35) -> /MCU/UART_RX
- U1 pad 61: unconnected-(U1-09-Pad61) -> GND
- U1 pad 66: unconnected-(U1-14-Pad66) -> GND
- U1 pad 69: unconnected-(U1-17-Pad69) -> GND
- U1 pad 73: unconnected-(U1-21-Pad73) -> GND
- U1 pad 74: unconnected-(U1-22-Pad74) -> GND
- U1 pad 75: unconnected-(U1-23-Pad75) -> /PC104_stack/12VA
- U1 pad 76: unconnected-(U1-24-Pad76) -> /PC104_stack/12VA
- U1 pad 77: unconnected-(U1-25-Pad77) -> +5V
- U1 pad 78: unconnected-(U1-26-Pad78) -> +5V
- U1 pad 79: unconnected-(U1-27-Pad79) -> +3V3
- U1 pad 80: unconnected-(U1-28-Pad80) -> +3V3
- U1 pad 81: unconnected-(U1-29-Pad81) -> GND
- U1 pad 82: unconnected-(U1-30-Pad82) -> GND
- U1 pad 84: unconnected-(U1-32-Pad84) -> GND
- U1 pad 97: unconnected-(U1-45-Pad97) -> /12V Power Supply/VBAT
- U1 pad 98: unconnected-(U1-46-Pad98) -> /12V Power Supply/VBAT
- U1 pad 99: unconnected-(U1-47-Pad99) -> GND
- U2 pad 1: unconnected-(U2-PE2-Pad1) -> /MCU/Valve9
- U2 pad 10: Net-(U2-VSS-Pad10) -> GND
- U2 pad 100: unconnected-(U2-VDD-Pad100) -> +3V3
- U2 pad 11: unconnected-(U2-VDD-Pad11) -> +3V3
- U2 pad 15: unconnected-(U2-PC0-Pad15) -> /MCU/I2C3_SCL
- U2 pad 16: unconnected-(U2-PC1-Pad16) -> /MCU/I2C3_SDA
- U2 pad 19: unconnected-(U2-VSSA-Pad19) -> GND
- U2 pad 2: unconnected-(U2-PE3-Pad2) -> /MCU/Valve10
- U2 pad 20: unconnected-(U2-VREF--Pad20) -> GND
- U2 pad 21: unconnected-(U2-VREF+-Pad21) -> +3V3
- U2 pad 22: unconnected-(U2-VDDA-Pad22) -> +3V3
- U2 pad 24: unconnected-(U2-PA1-Pad24) -> /MCU/Valve14
- U2 pad 25: unconnected-(U2-PA2-Pad25) -> /MCU/Valve15
- U2 pad 27: Net-(U2-VSS-Pad10) -> GND
- U2 pad 28: unconnected-(U2-VDD-Pad28) -> +3V3
- U2 pad 3: unconnected-(U2-PE4-Pad3) -> /MCU/Valve11
- U2 pad 33: unconnected-(U2-PC4-Pad33) -> /MCU/UART_TX
- U2 pad 34: unconnected-(U2-PC5-Pad34) -> /MCU/UART_RX
- U2 pad 4: unconnected-(U2-PE5-Pad4) -> /MCU/Valve12
- U2 pad 47: unconnected-(U2-PB10-Pad47) -> /MCU/I2C4_SCL
- U2 pad 48: unconnected-(U2-PB11-Pad48) -> /MCU/I2C4_SDA
- U2 pad 49: Net-(U2-VSS-Pad10) -> GND
- U2 pad 5: unconnected-(U2-PE6-Pad5) -> /MCU/Valve13
- U2 pad 50: unconnected-(U2-VDD-Pad50) -> +3V3
- U2 pad 51: unconnected-(U2-PB12-Pad51) -> /MCU/Valve1
- U2 pad 52: unconnected-(U2-PB13-Pad52) -> /MCU/I2C2_SCL
- U2 pad 53: unconnected-(U2-PB14-Pad53) -> /MCU/I2C2_SDA
- U2 pad 61: unconnected-(U2-PD14-Pad61) -> /MCU/Valve2
- U2 pad 62: unconnected-(U2-PD15-Pad62) -> /MCU/Valve3
- U2 pad 63: unconnected-(U2-PC6-Pad63) -> /MCU/Valve6
- U2 pad 64: unconnected-(U2-PC7-Pad64) -> /MCU/Valve5
- U2 pad 65: unconnected-(U2-PC8-Pad65) -> /MCU/Valve7
- U2 pad 66: unconnected-(U2-PC9-Pad66) -> /MCU/Valve8
- U2 pad 67: unconnected-(U2-PA8-Pad67) -> /MCU/Valve4
- U2 pad 70: unconnected-(U2-PA11-Pad70) -> /MCU/Valve16
- U2 pad 71: unconnected-(U2-PA12-Pad71) -> /MCU/Valve17
- U2 pad 72: unconnected-(U2-PA13-Pad72) -> /MCU/Valve18
- U2 pad 74: Net-(U2-VSS-Pad10) -> GND
- U2 pad 75: unconnected-(U2-VDD-Pad75) -> +3V3
- U2 pad 95: unconnected-(U2-PB8-Pad95) -> /MCU/I2C1_SCL
- U2 pad 96: unconnected-(U2-PB9-Pad96) -> /MCU/I2C1_SDA
- U2 pad 99: Net-(U2-VSS-Pad10) -> GND
