File: hw/PIB/monarch_payload_interface_board_rev1/_autosave-monarch_payload_interface_board_rev1.kicad_pcb (KiCad board)
At the start: 4 copper layers, 96 x 89.9 mm, 187 parts, among them J1 5037630291, J10 5037630491, J11 5037630691, J12 5037630691, J13 5037630491, J14 5037630491, J15 5037630691, J16 20021121-00008C4LF, J2 5037630291, J3 5037630691, J4 5037630691, J5 5037630691, J6 5037630691, J7 5037630691, J8 5037630691, J9 5037630491, Q1 FZT600TA, Q10 FZT600TA, Q11 FZT600TA, Q12 FZT600TA, Q13 FZT600TA, Q14 FZT600TA, Q15 FZT600TA, Q16 FZT600TA, Q17 FZT600TA, Q18 FZT600TA, Q19 FZT600TA, Q2 FZT600TA, Q3 FZT600TA, Q4 FZT600TA, Q5 FZT600TA, Q6 FZT600TA, Q7 FZT600TA, Q8 FZT600TA, Q9 FZT600TA, U1 Payload, U10 AD7124-8BCPZ-RL, U11 WSK06121L000FEA, U12 WSK06121L000FEA, U13 WSK06121L000FEA, U14 WSK06121L000FEA, U2 STM32L4A6VGTx, U3 MAX31856MUD_T, U4 TPS61088QRHLRQ1, U5 MAX31856MUD_T, U6 MAX31856MUD_T, U7 MAX31856MUD_T, U8 MAX31856MUD_T, U9 AD7124-8BCPZ-RL

Commit message: more minor tweaks
Parts:
- R49: value 1k -> 125
Changed lines of the file:
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@@
 			)
 		)
-		(property "Value" "1k"
+		(property "Value" "125"
 			(at 0 1.43 90)
 			(layer "F.Fab")
