File: hw/PIB/monarch_payload_interface_board_rev1/_autosave-MCU.kicad_sch (KiCad schematic)
At the start: 24 parts, among them J15 Conn_01x08_Pin, J16 SBH11-NBPC-D10-SM-BK, U2 STM32L4A6VGTx

Commit message: PIB Progress
Most MCU pins selected. more to come.
Parts:
- removed R25, R26: 4.7k, Resistor_SMD:R_0603_1608Metric, symbol Device:R_Small
Connections:
- net I2C2_SCL is gone; now on net Valve2: U2.52 (PB13)
- net I2C2_SDA is gone; now on net Valve3: U2.53 (PB14)
- net SPI3_MISO is gone; now on net Valve14: U2.79 (PC11)
- net SPI3_MOSI is gone; now on net Valve16: U2.80 (PC12)
- net SPI3_SCK is gone; now on net Valve13: U2.78 (PC10)
- net EN: now also U2.12 (PH0); no longer U2.68 (PA9)
- net Valve10: now also U2.65 (PC8); no longer U2.2 (PE3)
- net Valve11: now also U2.66 (PC9); no longer U2.3 (PE4)
- net Valve12: now also U2.67 (PA8); no longer U2.4 (PE5)
- net Valve13: no longer U2.5 (PE6)
- net Valve14: no longer U2.24 (PA1)
- net Valve15: now also U2.83 (PD2); no longer U2.25 (PA2)
- net Valve16: no longer U2.70 (PA11)
- net Valve17: now also U2.81 (PD0); no longer U2.71 (PA12)
- net Valve2: no longer U2.61 (PD14)
- net Valve3: no longer U2.62 (PD15)
- net Valve4: now also U2.63 (PC6); no longer U2.67 (PA8)
- net Valve5: now also U2.54 (PB15); no longer U2.64 (PC7)
- net Valve6: now also U2.40 (PE9); no longer U2.63 (PC6)
- net Valve7: now also U2.55 (PD8); no longer U2.65 (PC8)
- net Valve8: now also U2.56 (PD9); no longer U2.66 (PC9)
- net Valve9: now also U2.64 (PC7); no longer U2.1 (PE2)
- net at R49.2: no longer U2.81 (PD0)
- net SPI2_SCK: now reaches U2.82 (PD1)
- net SPI2_MISO: now reaches U2.84 (PD3)
- net SPI2_MOSI: now reaches U2.85 (PD4)
Other:
- moved on the sheet: C17, C18, D1, R49
