File: hw/PIB/monarch_payload_interface_board_rev1/_autosave-connectors.kicad_sch (KiCad schematic)
At the start: 14 parts, among them J1 5037630291, J10 5037630491, J11 5037630691, J12 5037630691, J13 5037630491, J14 5037630491, J2 5037630291, J3 5037630691, J4 5037630691, J5 5037630691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

Commit message: PIB Progress
Most MCU pins selected. more to come.
Connections:
- net T1+: now also J8.4; no longer J8.3
- net T1-: now also J8.3; no longer J8.4
- net T2+: now also J8.6; no longer J8.5
- net T2-: now also J8.5; no longer J8.6
- net T3+: now also J9.2; no longer J9.1
- net T3-: now also J9.1; no longer J9.2
- net T4+: now also J9.4; no longer J9.3
- net T4-: now also J9.3; no longer J9.4
