File: hw/PIB/monarch_payload_interface_board_rev1/MCU.kicad_sch (KiCad schematic)
At the start: 24 parts, among them J15 Conn_01x08_Pin, J16 SBH11-NBPC-D10-SM-BK, U2 STM32L4A6VGTx

Commit message: PIB layout update
done pending Ben O approval
Parts:
- removed J15: Conn_01x08_Pin, symbol Connector:Conn_01x08_Pin
- removed J16: SBH11-NBPC-D10-SM-BK, SBH11:CONN_SBH11-NBPC-D10-SM-BK_SUL, symbol SBH11:SBH11-NBPC-D10-SM-BK
- removed R22, R25, R26, R27, R28, R29: 4.7k, Resistor_SMD:R_0603_1608Metric, symbol Device:R_Small
- added J16: 20021121-00008C4LF, 20021121:AMPHENOL_20021121-00008C4LF, symbol 20021121:20021121-00008C4LF
Connections:
- net I2C1_SDA is gone; now on net T1: U2.96 (PB9)
- net I2C2_SCL is gone; now on net Valve2: U2.52 (PB13)
- net I2C2_SDA is gone; now on net Valve3: U2.53 (PB14)
- net SPI3_MISO is gone; now on net Valve14: U2.79 (PC11)
- net SPI3_MOSI is gone; now on net Valve16: U2.80 (PC12)
- net SPI3_SCK is gone; now on net Valve13: U2.78 (PC10)
- net +3V3: now also J16.1
- net EN: now also U2.12 (PH0); no longer U2.68 (PA9)
- net GND: now also J16.8
- net Heater0: now also U2.69 (PA10); no longer U2.35 (PB0)
- net JTCK: now also J16.5
- net JTDI: now also J16.3
- net JTDO: now also J16.6
- net JTMS: now also J16.4
- net NJTRST: now also J16.2
- net NRST: now also J16.7
- net PT: now also U2.3 (PE4); no longer U2.26 (PA3)
- net T1: no longer U2.41 (PE10)
- net T2: now also U2.2 (PE3); no longer U2.42 (PE11)
- net T3: now also U2.97 (PE0); no longer U2.43 (PE12)
- net T4: now also U2.1 (PE2); no longer U2.44 (PE13)
- net T5: now also U2.98 (PE1); no longer U2.45 (PE14)
- net Valve10: now also U2.65 (PC8); no longer U2.2 (PE3)
- net Valve11: now also U2.66 (PC9); no longer U2.3 (PE4)
- net Valve12: now also U2.67 (PA8); no longer U2.4 (PE5)
- net Valve13: no longer U2.5 (PE6)
- net Valve14: no longer U2.24 (PA1)
- net Valve15: now also U2.83 (PD2); no longer U2.25 (PA2)
- net Valve16: no longer U2.70 (PA11)
- net Valve17: now also U2.81 (PD0); no longer U2.71 (PA12)
- net Valve18: now also U2.70 (PA11); no longer U2.69 (PA10)
- net Valve2: no longer U2.61 (PD14)
- net Valve3: no longer U2.62 (PD15)
- net Valve4: now also U2.63 (PC6); no longer U2.67 (PA8)
- net Valve5: now also U2.54 (PB15); no longer U2.64 (PC7)
- net Valve6: now also U2.40 (PE9); no longer U2.63 (PC6)
- net Valve7: now also U2.55 (PD8); no longer U2.65 (PC8)
- net Valve8: now also U2.56 (PD9); no longer U2.66 (PC9)
- net Valve9: now also U2.64 (PC7); no longer U2.1 (PE2)
- net at U2.46 (PE15): now also R49.2
- net SPI2_SCK: now reaches U2.82 (PD1)
- net SPI2_MISO: now reaches U2.84 (PD3)
- net SPI2_MOSI: now reaches U2.85 (PD4)
- net I2C1_SCL: no longer names the net of U2.95 (PB8)
- net I2C3_SCL: no longer names the net of U2.15 (PC0)
- net I2C3_SDA: no longer names the net of U2.16 (PC1)
Other:
- moved on the sheet: C17, C18, D1, R23, R24, R49

Commit message: PIB minor updates & radio board
Connections:
- net UART4_TX: now reaches U2.23 (PA0)
- net UART4_RX: now reaches U2.24 (PA1)
- net UART_RX renamed USART3_RX
- net UART_TX renamed USART3_TX
Changed lines of the file:
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@@
+	(wire
+		(pts
+			(xy 153.67 48.26) (xy 156.21 48.26)
+		)
+		(stroke
+			(width 0)
+			(type default)
+		)
+	)
 	(wire
 		(pts
@@
 	(wire
 		(pts
-			(xy 153.67 55.88) (xy 156.21 55.88)
-		)
-		(stroke
-			(width 0)
-			(type default)
-		)
-	)
-	(wire
-		(pts
 			(xy 105.41 73.66) (xy 107.95 73.66)
 		)
@@
 	(wire
 		(pts
-			(xy 156.21 41.91) (xy 156.21 43.18)
-		)
-		(stroke
-			(width 0)
-			(type default)
-		)
-	)
-	(wire
-		(pts
 			(xy 63.5 83.82) (xy 68.58 83.82)
 		)
@@
 		(pts
 			(xy 156.21 35.56) (xy 173.99 35.56)
-		)
-		(stroke
-			(width 0)
-			(type default)
-		)
-	)
-	(wire
-		(pts
-			(xy 153.67 53.34) (xy 156.21 53.34)
 		)
 		(stroke
@@
 		)
 	)
+	(hierarchical_label "UART4_TX"
+		(shape output)
+		(at 156.21 48.26 0)
+		(effects
+			(font
+				(size 1.27 1.27)
+			)
+			(justify left)
+		)
+	)
 	(hierarchical_label "Valve6"
 		(shape output)
@@
 		)
 	)
-	(hierarchical_label "UART_TX"
+	(hierarchical_label "USART3_TX"
 		(shape output)
 		(at 156.21 144.78 0)
@@
 		)
 	)
-	(hierarchical_label "UART_RX"
+	(hierarchical_label "USART3_RX"
 		(shape input)
 		(at 156.21 147.32 0)
@@
 		(shape output)
 		(at 156.21 154.94 0)
+		(effects
+			(font
+				(size 1.27 1.27)
+			)
+			(justify left)
+		)
+	)
+	(hierarchical_label "UART4_RX"
+		(shape input)
+		(at 156.21 50.8 0)
 		(effects
 			(font
@@
 	(symbol
 		(lib_id "power:GND")
-		(at 156.21 43.18 0)
+		(at 156.21 41.91 0)
 		(unit 1)
 		(exclude_from_sim no)
@@
 		(dnp no)
 		(property "Reference" "#PWR041"
-			(at 156.21 49.53 0)
+			(at 156.21 48.26 0)
 			(effects
 				(font
@@
 		)
 		(property "Value" "GND"
-			(at 156.21 46.736 0)
+			(at 156.21 45.466 0)
 			(effects
 				(font
@@
 		)
 		(property "Footprint" ""
-			(at 156.21 43.18 0)
+			(at 156.21 41.91 0)
 			(effects
 				(font
@@
 		)
 		(property "Datasheet" ""
-			(at 156.21 43.18 0)
+			(at 156.21 41.91 0)
 			(effects
 				(font
@@
 		)
 		(property "Description" "Power symbol creates a global label with name \"GND\" , ground"
-			(at 156.21 43.18 0)
-			(effects
-				(font
+			(at 156.21 41.91 0)
+			(effects
+				(font

Commit message: minor tweaks
Parts:
- R49: value 1k -> 125
Changed lines of the file:
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@@
-		)
-	)
-	(hierarchical_label "EN"
-		(shape output)
-		(at 156.21 -27.94 0)
-		(effects
-			(font
-				(size 1.27 1.27)
-			)
-			(justify left)
 		)
 	)
@@
 			)
 		)
-		(property "Value" "1k"
+		(property "Value" "125"
 			(at 100.33 106.68 90)
 			(effects

Commit message: Software/Hardware
Connections:
- net GND: now also U2.94 (PH3)
