File: hw/PIB/monarch_payload_interface_board_rev1/heater.kicad_sch (KiCad schematic)
At the start: 3 parts, among them Q19 FZT600TA

Commit message: PCB updates
Parts:
- removed CR19: S1J-13-F, s1j:SMA_DIO-L, symbol s1j:S1J-13-F
- R40: footprint Resistor_SMD:R_0402_1005Metric -> Resistor_SMD:R_0603_1608Metric
Connections:
- net Heater0- renamed +12VA

Commit message: PIB Progress
Most MCU pins selected. more to come.
Connections:
- net +12VA: no longer Q19.2 (C_1), Q19.4 (C_2)
- new net Heater0-: Q19.2 (C_1), Q19.4 (C_2)
Changed lines of the file:
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@@
 	)
 	(junction
-		(at 157.48 101.6)
+		(at 148.59 101.6)
 		(diameter 0)
 		(color 0 0 0 0)
 	)
-	(junction
-		(at 151.13 85.09)
-		(diameter 0)
-		(color 0 0 0 0)
-	)
-	(junction
-		(at 144.78 101.6)
-		(diameter 0)
-		(color 0 0 0 0)
-	)
-	(wire
-		(pts
-			(xy 137.16 101.6) (xy 144.78 101.6)
+	(wire
+		(pts
+			(xy 137.16 101.6) (xy 148.59 101.6)
 		)
 		(stroke
@@
 	(wire
 		(pts
-			(xy 157.48 101.6) (xy 163.83 101.6)
-		)
-		(stroke
-			(width 0)
-			(type default)
-		)
-	)
-	(wire
-		(pts
-			(xy 144.78 85.09) (xy 151.13 85.09)
-		)
-		(stroke
-			(width 0)
-			(type default)
-		)
-	)
-	(wire
-		(pts
 			(xy 125.73 74.93) (xy 137.16 74.93)
 		)
@@
 	(wire
 		(pts
-			(xy 151.13 85.09) (xy 157.48 85.09)
-		)
-		(stroke
-			(width 0)
-			(type default)
-		)
-	)
-	(wire
-		(pts
-			(xy 157.48 85.09) (xy 157.48 88.9)
+			(xy 148.59 88.9) (xy 148.59 93.98)
 		)
 		(stroke
@@
 	(wire
 		(pts
-			(xy 157.48 99.06) (xy 157.48 101.6)
-		)
-		(stroke
-			(width 0)
-			(type default)
-		)
-	)
-	(wire
-		(pts
-			(xy 144.78 85.09) (xy 144.78 101.6)
+			(xy 148.59 101.6) (xy 163.83 101.6)
+		)
+		(stroke
+			(width 0)
+			(type default)
+		)
+	)
+	(wire
+		(pts
+			(xy 148.59 99.06) (xy 148.59 101.6)
 		)
 		(stroke
@@
 	(wire
 		(pts
-			(xy 151.13 83.82) (xy 151.13 85.09)
-		)
-		(stroke
-			(width 0)
-			(type default)
-		)
-	)
-	(wire
-		(pts
 			(xy 127 106.68) (xy 130.81 106.68)
-		)
-		(stroke
-			(width 0)
-			(type default)
-		)
-	)
-	(wire
-		(pts
-			(xy 144.78 101.6) (xy 157.48 101.6)
 		)
 		(stroke
@@
 	(hierarchical_label "Heater0+"
 		(shape output)
-		(at 157.48 88.9 0)
+		(at 148.59 93.98 0)
 		(effects
 			(font
@@
 	(hierarchical_label "Heater0-"
 		(shape input)
-		(at 157.48 99.06 0)
+		(at 148.59 99.06 0)
 		(effects
 			(font
@@
 	(symbol
 		(lib_id "power:+3V3")
-		(at 151.13 83.82 0)
+		(at 148.59 88.9 0)
 		(unit 1)
 		(exclude_from_sim no)
@@
 		(dnp no)
 		(property "Reference" "#PWR0212"
-			(at 151.13 87.63 0)
+			(at 148.59 92.71 0)
 			(effects
 				(font
@@
 		)
 		(property "Value" "+12VA"
-			(at 146.558 82.042 0)
+			(at 144.018 87.122 0)
 			(effects
 				(font
@@
 		)
 		(property "Footprint" ""
-			(at 151.13 83.82 0)
+			(at 148.59 88.9 0)
 			(effects
 				(font
@@
 		)
 		(property "Datasheet" ""
-			(at 151.13 83.82 0)
+			(at 148.59 88.9 0)
 			(effects
 				(font
@@
 		)
 		(property "Description" "Power symbol creates a global label with name \"+3V3\""
-			(at 151.13 83.82 0)
-			(effects
-				(font
+			(at 148.59 88.9 0)
+			(effects
+				(font
