File: hw/PIB/monarch_payload_interface_board_rev1/power supply.kicad_sch (KiCad schematic)
At the start: 17 parts, among them U4 TPS61088QRHLRQ1

Commit message: Schematic Review
Parts:
- removed L1: XEL4020-561MEC, XEL:IND_XEL4020_COC-L, symbol XEL:XEL4020-561MEC
- added L1: EXLA1V0402-R82-R, EXLA1V0402-R82-R:IND_EXLA1V0402-R82-R, symbol EXLA1V0402-R82-R:EXLA1V0402-R82-R
Connections:
- net GND: now also C10.2
- net VBAT: now also C9.1, L1.1
- net at C1.2, R17.1, U4.4 (SW)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: now also L1.2
Other:
- moved on the sheet: C10

Commit message: PCB updates
Parts:
- removed C2: 82uF, 35SVT82M:CAP_35SVT82M, symbol 35SVT82M:35SVT82M
- added C2, C51, C52: 22u, Capacitor_SMD:C_0805_2012Metric, symbol Device:C_Small
- added C53: 15u, Capacitor_SMD:C_1206_3216Metric, symbol Device:C_Small
- added C54: 1u, Capacitor_SMD:C_0603_1608Metric, symbol Device:C_Small
- added R46, R55: 100k, Resistor_SMD:R_0603_1608Metric, symbol Device:R_Small
- added R47, R48: 300k, Resistor_SMD:R_0603_1608Metric, symbol Device:R_Small
- added U14: WSK06121L000FEA, WSK:SMT_121L000FEA_VIS, symbol WSK:WSK06121L000FEA
- C1: value 100nF -> 0.1u
- C10, C9: footprint Capacitor_SMD:C_0603_1608Metric -> Capacitor_SMD:C_0805_2012Metric
- C3: footprint Capacitor_SMD:C_0603_1608Metric -> Capacitor_SMD:C_1206_3216Metric
- R17, R18, R19, R20, R21: footprint Resistor_SMD:R_0402_1005Metric -> Resistor_SMD:R_0603_1608Metric
Connections:
- net GND: now also U4.13 (MODE), C2.2, C51.2, C52.2, C53.2, C54.2, R46.1, R55.1
- net at C7.2, U4.1 (VCC): no longer U4.2 (EN)
- net 12VB: no longer names the net of C3.1, R18.1, U4.14 (VOUT), U4.15 (VOUT), U4.16 (VOUT)
- net 12VB: now also C2.1, C51.1, C52.1, C53.1, C54.1, U14.I1
- new net: R47.2, U14.E1
- new net: R48.2, U14.E2
- new net +12VB: U14.I2
- new net 12VB_VA: R46.2, R47.1
- new net 12VB_VB: R48.1, R55.2
- new net EN: U4.2 (EN)
Other:
- moved on the sheet: C3
