File: hw/PIB/monarch_payload_interface_board_rev2/connectors.kicad_sch (KiCad schematic)
At the start: 18 parts, among them J1 2200980271, J13 2200980471, J14 5037630491, J15 5037630491, J16 2200980271, J18 2200980671, J19 2200980671, J2 Conn_01x06, J20 2200980671, J21 2200980671, J22 2200980671, J23 2200980671, J24 2200980671, J25 5037630491, J3 Conn_01x05, J4 Conn_01x04, J6 2200980671, J8 5037630691

Commit message: AD7124 fixes
Parts:
- added J5: Conn_01x05, Connector_PinHeader_1.00mm:PinHeader_1x05_P1.00mm_Vertical, symbol Connector_Generic:Conn_01x05
- J2: footprint Connector_PinHeader_1.27mm:PinHeader_1x06_P1.27mm_Vertical -> (none)
Connections:
- net *DRDY: now also J5.5 (Pin_5); no longer J2.5 (Pin_5)
- net *FAULT: now also J5.4 (Pin_4); no longer J2.4 (Pin_4)
- net SPI2_MISO: now also J5.1 (Pin_1); no longer J2.1 (Pin_1)
- net SPI2_MOSI: now also J5.2 (Pin_2); no longer J2.2 (Pin_2)
- net SPI2_SCK: now also J5.3 (Pin_3); no longer J2.3 (Pin_3)
- net T1: now also J2.5 (Pin_5); no longer J2.6 (Pin_6)
- new net PT: J2.6 (Pin_6)
- new net T2: J2.4 (Pin_4)
- new net T3: J2.3 (Pin_3)
- new net T4: J2.2 (Pin_2)
- new net T5: J2.1 (Pin_1)
Other:
- note added: "Chip Select Connector"
- note removed: "AD7124-8 Pressure Connector"
- moved on the sheet: J1, J13, J14, J15, J16, J18, J19, J20, J21, J22, J23, J24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

Commit message: Schematic Updates Finished -> AD7124 Voltage Reading Fix + Connector Linkage Issue Fix
Connections:
- net UART4_RX is gone; now on net UART_PPU_TX: J4.1 (Pin_1)
- net UART4_TX is gone; now on net UART_PPU_RX: J4.2 (Pin_2)
Changed lines of the file:
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@@
-		)
-	)
-	(hierarchical_label "UART4_RX"
-		(shape input)
-		(at 92.71 77.47 180)
-		(effects
-			(font
-				(size 1.27 1.27)
-			)
-			(justify right)
 		)
 	)
@@
 		)
 	)
+	(hierarchical_label "UART_PPU_TX"
+		(shape output)
+		(at 92.71 77.47 180)
+		(effects
+			(font
+				(size 1.27 1.27)
+			)
+			(justify right)
+		)
+	)
 	(hierarchical_label "USART3_TX"
 		(shape output)
@@
 		)
 	)
+	(hierarchical_label "UART_PPU_RX"
+		(shape input)
+		(at 92.71 80.01 180)
+		(effects
+			(font
+				(size 1.27 1.27)
+			)
+			(justify right)
+		)
+	)
 	(hierarchical_label "Valve3-"
 		(shape output)
@@
 		(effects
 			(font
-				(size 1.27 1.27)
-			)
-			(justify right)
-		)
-	)
-	(hierarchical_label "UART4_TX"
-		(shape output)
-		(at 92.71 80.01 180)
-		(effects
-			(font

Commit message: Footprint Selected
Parts:
- J14, J15, J25: value 5037630491 -> 2200980471; footprint CONN_5037630000-SD_04_MOL -> Connector_Molex_Micro-Lock-Plus:Molex_Micro-Lock_2200980471_1x04_P1.25mm_Horizontal
- J2: footprint (none) -> Connector_PinHeader_2.54mm:PinHeader_1x06_P2.54mm_Vertical
- J3, J5: footprint Connector_PinHeader_1.00mm:PinHeader_1x05_P1.00mm_Vertical -> Connector_PinHeader_2.54mm:PinHeader_1x05_P2.54mm_Vertical
- J4: footprint Connector_PinHeader_1.00mm:PinHeader_1x04_P1.00mm_Vertical -> Connector_PinHeader_2.54mm:PinHeader_1x04_P2.54mm_Vertical
- J8: value 5037630691 -> 2200980671; footprint CONN_5037630000-SD_06_MOL -> Connector_Molex_Micro-Lock-Plus:Molex_Micro-Lock_2200980671_1x06_P1.25mm_Horizontal
Changed lines of the file:
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@@
-		(lib_name "5037630491_3")
-		(lib_id "5037630491:5037630491")
-		(at 194.31 87.63 0)
-		(unit 1)
-		(body_style 1)
-		(exclude_from_sim no)
-		(in_bom yes)
-		(on_board yes)
-		(in_pos_files yes)
-		(dnp no)
-		(fields_autoplaced yes)
-		(property "Reference" "J15"
-			(at 208.28 90.1699 0)
-			(show_name no)
-			(do_not_autoplace no)
-			(effects
-				(font
-					(size 1.524 1.524)
-				)
-				(justify left)
-			)
-		)
-		(property "Value" "5037630491"
-			(at 208.28 92.7099 0)
-			(show_name no)
-			(do_not_autoplace no)
-			(effects
-				(font
-					(size 1.524 1.524)
-				)
-				(justify left)
-			)
-		)
-		(property "Footprint" "CONN_5037630000-SD_04_MOL"
-			(at 194.31 87.63 0)
-			(hide yes)
-			(show_name no)
-			(do_not_autoplace no)
-			(effects
-				(font
-					(size 1.27 1.27)
-					(italic yes)
-				)
-			)
-		)
-		(property "Datasheet" "https://www.molex.com/en-us/products/part-detail-pdf/5037630491?display=pdf"
-			(at 194.31 87.63 0)
-			(hide yes)
-			(show_name no)
-			(do_not_autoplace no)
-			(effects
-				(font
-					(size 1.27 1.27)
-					(italic yes)
-				)
-			)
-		)
-		(property "Description" ""
-			(at 194.31 87.63 0)
-			(hide yes)
-			(show_name no)
-			(do_not_autoplace no)
-			(effects
-				(font
-					(size 1.27 1.27)
-				)
-			)
-		)
-		(pin "4"
-		)
-		(pin "2"
-		)
-		(pin "3"
-		)
-		(pin "1"
-		)
-		(instances
-			(project "monarch_payload_interface_board_rev2"
-				(path "/bf7ee58d-ac53-49d1-a6b2-96a87d67b737/ef907aa1-ebae-4134-aea0-07912ab07993"
-					(reference "J15")
-					(unit 1)
-				)
-			)
-		)
-	)
-	(symbol
 		(lib_name "5037630491_3")
 		(lib_id "5037630491:5037630491")
@@
 			)
 		)
-		(property "Value" "5037630491"
+		(property "Value" "2200980471"
 			(at 55.88 93.9799 0)
 			(show_name no)
@@
 			)
 		)
-		(property "Footprint" "CONN_5037630000-SD_04_MOL"
+		(property "Footprint" "Connector_Molex_Micro-Lock-Plus:Molex_Micro-Lock_2200980471_1x04_P1.25mm_Horizontal"
 			(at 41.91 88.9 0)
 			(hide yes)
@@
 			)
 		)
-		(property "Datasheet" "https://www.molex.com/en-us/products/part-detail-pdf/5037630491?display=pdf"
+		(property "Datasheet" "https://www.molex.com/en-us/products/part-detail/2200980471"
 			(at 41.91 88.9 0)
 			(hide yes)
@@
 			)
 		)
-		(property "Footprint" "Connector_PinHeader_1.00mm:PinHeader_1x05_P1.00mm_Vertical"
+		(property "Footprint" "Connector_PinHeader_2.54mm:PinHeader_1x05_P2.54mm_Vertical"
 			(at 146.05 73.66 0)
 			(hide yes)
@@
 			)
 		)
-		(property "Footprint" "Connector_PinHeader_1.00mm:PinHeader_1x04_P1.00mm_Vertical"
+		(property "Footprint" "Connector_PinHeader_2.54mm:PinHeader_1x04_P2.54mm_Vertical"
 			(at 97.79 80.01 0)
 			(hide yes)
@@
 	)
 	(symbol
+		(lib_name "5037630491_2")
+		(lib_id "5037630491:5037630491")
+		(at 247.65 38.1 0)
+		(unit 1)
+		(body_style 1)
+		(exclude_from_sim no)
+		(in_bom yes)
+		(on_board yes)
+		(in_pos_files yes)
+		(dnp no)
+		(fields_autoplaced yes)
+		(property "Reference" "J25"
+			(at 261.62 40.6399 0)
+			(show_name no)
+			(do_not_autoplace no)
+			(effects
+				(font
+					(size 1.524 1.524)
+				)
+				(justify left)
+			)
+		)
+		(property "Value" "2200980471"
+			(at 261.62 43.1799 0)
+			(show_name no)
+			(do_not_autoplace no)
+			(effects
+				(font
+					(size 1.524 1.524)
+				)
+				(justify left)
+			)
+		)
+		(property "Footprint" "Connector_Molex_Micro-Lock-Plus:Molex_Micro-Lock_2200980471_1x04_P1.25mm_Horizontal"
+			(at 247.65 38.1 0)
+			(hide yes)
+			(show_name no)
+			(do_not_autoplace no)
+			(effects
+				(font
+					(size 1.27 1.27)
+					(italic yes)
+				)
+			)
+		)
+		(property "Datasheet" "https://www.molex.com/en-us/products/part-detail/2200980471"
+			(at 247.65 38.1 0)
+			(hide yes)
+			(show_name no)
+			(do_not_autoplace no)
+			(effects
+				(font
+					(size 1.27 1.27)
+					(italic yes)
+				)
+			)
+		)
+		(property "Description" ""
+			(at 247.65 38.1 0)
+			(hide yes)
+			(show_name no)
+			(do_not_autoplace no)
+			(effects
+				(font
+					(size 1.27 1.27)
+				)
+			)
+		)
+		(pin "4"
+		)
+		(pin "2"
+		)
+		(pin "1"
+		)
+		(pin "3"
+		)
+		(instances
+			(project "monarch_payload_interface_board_rev2"
+				(path "/bf7ee58d-ac53-49d1-a6b2-96a87d67b737/ef907aa1-ebae-4134-aea0-07912ab07993"
+					(reference "J25")
+					(unit 1)
+				)
+			)
+		)
+	)
+	(symbol
 		(lib_id "Connector_Generic:Conn_01x05")
 		(at 146.05 93.98 0)
@@
 			)
 		)
-		(property "Footprint" "Connector_PinHeader_1.00mm:PinHeader_1x05_P1.00mm_Vertical"
+		(property "Footprint" "Connector_PinHeader_2.54mm:PinHeader_1x05_P2.54mm_Vertical"
 			(at 146.05 93.98 0)
 			(hide yes)
@@
 	)
 	(symbol
-		(lib_name "5037630491_3")
-		(lib_id "5037630491:5037630491")
-		(at 247.65 38.1 0)
-		(unit 1)
-		(body_style 1)
-		(exclude_from_sim no)
-		(in_bom yes)
-		(on_board yes)
-		(in_pos_files yes)
-		(dnp no)
-		(fields_autoplaced yes)
-		(property "Reference" "J25"
-			(at 261.62 40.6399 0)
-			(show_name no)
-			(do_not_autoplace no)
-			(effects
-				(font
-					(size 1.524 1.524)
-				)
-				(justify left)
-			)
-		)
-		(property "Value" "5037630491"
-			(at 261.62 43.1799 0)
-			(show_name no)
-			(do_not_autoplace no)
-			(effects
-				(font
-					(size 1.524 1.524)
-				)
-				(justify left)
-			)
-		)
-		(property "Footprint" "CONN_5037630000-SD_04_MOL"
-			(at 247.65 38.1 0)
-			(hide yes)
-			(show_name no)
-			(do_not_autoplace no)
-			(effects
-				(font
-					(size 1.27 1.27)
-					(italic yes)
-				)
-			)
-		)
-		(property "Datasheet" "https://www.molex.com/en-us/products/part-detail-pdf/5037630491?display=pdf"
-			(at 247.65 38.1 0)
-			(hide yes)
-			(show_name no)
-			(do_not_autoplace no)
-			(effects
-				(font
-					(size 1.27 1.27)
-					(italic yes)
-				)
-			)
-		)
-		(property "Description" ""
-			(at 247.65 38.1 0)
-			(hide yes)
-			(show_name no)
-			(do_not_autoplace no)
-			(effects
-				(font
-					(size 1.27 1.27)
-				)
-			)
-		)
-		(pin "4"
-		)
-		(pin "2"
-		)
-		(pin "3"
-		)
-		(pin "1"
-		)
-		(instances
-			(project "monarch_payload_interface_board_rev2"
-				(path "/bf7ee58d-ac53-49d1-a6b2-96a87d67b737/ef907aa1-ebae-4134-aea0-07912ab07993"
-					(reference "J25")
-					(unit 1)
-				)
-			)
-		)
-	)
-	(symbol
 		(lib_id "power:GND")
 		(at 259.08 21.59 90)
@@
 			)
 		)
-		(property "Footprint" ""
+		(property "Footprint" "Connector_PinHeader_2.54mm:PinHeader_1x06_P2.54mm_Vertical"
 			(at 252.73 90.17 0)
 			(hide yes)
@@
 			)
 		)
-		(property "Value" "5037630691"
+		(property "Value" "2200980671"
 			(at 55.88 73.6599 0)
 			(show_name no)
@@
 			)
 		)
-		(property "Footprint" "CONN_5037630000-SD_06_MOL"
+		(property "Footprint" "Connector_Molex_Micro-Lock-Plus:Molex_Micro-Lock_2200980671_1x06_P1.25mm_Horizontal"
 			(at 41.91 66.04 0)
 			(hide yes)
@@
 			)
 		)
-		(property "Datasheet" "https://www.molex.com/en-us/products/part-detail-pdf/5037630691?display=pdf"
+		(property "Datasheet" "https://www.molex.com/en-us/products/part-detail/2200980671"
 			(at 41.91 66.04 0)
 			(hide yes)
@@
 					(unit 1)
 				)
+			)
+		)
+	)
+	(symbol
+		(lib_name "5037630491_2")
+		(lib_id "5037630491:5037630491")
+		(at 194.31 87.63 0)
+		(unit 1)
+		(body_style 1)
+		(exclude_from_sim no)
+		(in_bom yes)
+		(on_board yes)
+		(in_pos_files yes)
+		(dnp no)
+		(fields_autoplaced yes)
+		(property "Reference" "J15"
+			(at 208.28 90.1699 0)
+			(show_name no)
+			(do_not_autoplace no)
+			(effects
+				(font
+					(size 1.524 1.524)
+				)
+				(justify left)
+			)
+		)
+		(property "Value" "2200980471"
+			(at 208.28 92.7099 0)
+			(show_name no)
+			(do_not_autoplace no)
+			(effects
+				(font
+					(size 1.524 1.524)
+				)
+				(justify left)
+			)
+		)
+		(property "Footprint" "Connector_Molex_Micro-Lock-Plus:Molex_Micro-Lock_2200980471_1x04_P1.25mm_Horizontal"
+			(at 194.31 87.63 0)
+			(hide yes)
+			(show_name no)
+			(do_not_autoplace no)
+			(effects
+				(font
+					(size 1.27 1.27)
+					(italic yes)
+				)
+			)
+		)
+		(property "Datasheet" "https://www.molex.com/en-us/products/part-detail/2200980471"
+			(at 194.31 87.63 0)
+			(hide yes)
+			(show_name no)
+			(do_not_autoplace no)
+			(effects
+				(font
+					(size 1.27 1.27)
+					(italic yes)
+				)
+			)
+		)
+		(property "Description" ""
+			(at 194.31 87.63 0)
+			(hide yes)
+			(show_name no)
+			(do_not_autoplace no)
+			(effects
+				(font
+					(size 1.27 1.27)
+				)
+			)
+		)
+		(pin "4"
+		)
+		(pin "2"
+		)
+		(pin "1"
+		)
+		(pin "3"
+		)
+		(instances
+			(project "monarch_payload_interface_board_rev2"
+				(path "/bf7ee58d-ac53-49d1-a6b2-96a87d67b737/ef907aa1-ebae-4134-aea0-07912ab07993"
+					(reference "J15")
+					(unit 1)
+				)

Commit message: Initial Routing Work + Placement
Other:
- moved on the sheet: J24
Changed lines of the file:
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@@
 	(wire
 		(pts
-			(xy 242.57 63.5) (xy 247.65 63.5)
+			(xy 242.57 63.5) (xy 259.08 63.5)
 		)
 		(stroke
@@
 	(wire
 		(pts
+			(xy 259.08 71.12) (xy 247.65 71.12)
+		)
+		(stroke
+			(width 0)
+			(type default)
+		)
+	)
+	(wire
+		(pts
 			(xy 185.42 92.71) (xy 194.31 92.71)
 		)
@@
 	(wire
 		(pts
-			(xy 243.84 68.58) (xy 247.65 68.58)
+			(xy 243.84 68.58) (xy 259.08 68.58)
 		)
 		(stroke
@@
 	(wire
 		(pts
-			(xy 243.84 71.12) (xy 247.65 71.12)
-		)
-		(stroke
-			(width 0)
-			(type default)
-		)
-	)
-	(wire
-		(pts
 			(xy 33.02 52.07) (xy 41.91 52.07)
 		)
@@
 	(wire
 		(pts
-			(xy 243.84 58.42) (xy 247.65 58.42)
+			(xy 243.84 58.42) (xy 259.08 58.42)
 		)
 		(stroke
@@
 	(wire
 		(pts
-			(xy 242.57 66.04) (xy 247.65 66.04)
+			(xy 242.57 66.04) (xy 259.08 66.04)
 		)
 		(stroke
@@
 	(wire
 		(pts
-			(xy 243.84 60.96) (xy 247.65 60.96)
+			(xy 243.84 60.96) (xy 259.08 60.96)
 		)
 		(stroke
@@
 		(lib_name "5037630691_1")
 		(lib_id "5037630691:5037630691")
-		(at 247.65 58.42 0)
+		(at 259.08 58.42 0)
 		(unit 1)
 		(body_style 1)
@@
 		(fields_autoplaced yes)
 		(property "Reference" "J24"
-			(at 261.62 63.4999 0)
+			(at 273.05 63.4999 0)
 			(show_name no)
 			(do_not_autoplace no)
@@
 		)
 		(property "Value" "2200980671"
-			(at 261.62 66.0399 0)
+			(at 273.05 66.0399 0)
 			(show_name no)
 			(do_not_autoplace no)
@@
 		)
 		(property "Footprint" "Connector_Molex_Micro-Lock-Plus:Molex_Micro-Lock_2200980671_1x06_P1.25mm_Horizontal"
-			(at 247.65 58.42 0)
+			(at 259.08 58.42 0)
 			(hide yes)
 			(show_name no)
@@
 		)
 		(property "Datasheet" "https://www.molex.com/en-us/products/part-detail/2200980671"
-			(at 247.65 58.42 0)
+			(at 259.08 58.42 0)
 			(hide yes)
 			(show_name no)
@@
 		)
 		(property "Description" ""
-			(at 247.65 58.42 0)
+			(at 259.08 58.42 0)
 			(hide yes)
 			(show_name no)
@@
 	(symbol
 		(lib_id "power:+12VA")
-		(at 243.84 71.12 90)
+		(at 247.65 71.12 90)
 		(mirror x)
 		(unit 1)
@@
 		(in_pos_files yes)
 		(dnp no)
-		(fields_autoplaced yes)
 		(property "Reference" "#PWR0186"
-			(at 247.65 71.12 0)
+			(at 251.46 71.12 0)
 			(hide yes)
 			(show_name no)
@@
 		)
 		(property "Value" "+12VA"
-			(at 240.03 71.1201 90)
+			(at 244.348 70.866 90)
 			(show_name no)
 			(do_not_autoplace no)
@@
 		)
 		(property "Footprint" ""
-			(at 243.84 71.12 0)
+			(at 247.65 71.12 0)
 			(hide yes)
 			(show_name no)
@@
 		)
 		(property "Datasheet" ""
-			(at 243.84 71.12 0)
+			(at 247.65 71.12 0)
 			(hide yes)
 			(show_name no)
@@
 		)
 		(property "Description" "Power symbol creates a global label with name \"+12VA\""
-			(at 243.84 71.12 0)
+			(at 247.65 71.12 0)
 			(hide yes)
 			(show_name no)

Commit message: FINAL REVIEW DONE + A lot of fixes. DRC PASSED
Parts:
- added J7: Conn_01x02, Connector_PPU:CONN02_534260210_MOL, symbol Connector_Generic:Conn_01x02
Connections:
- net +12VA: now also J7.2 (Pin_2)
- net GND: now also J7.1 (Pin_1)
Other:
- note added: "PPU 12V Connector"
