File: hw/PIB/monarch_payload_interface_board_rev2/heater.kicad_sch (KiCad schematic)
At the start: 2 parts, among them Q19 FZT600TA

Commit message: Connector Additions
Other:
- moved on the sheet: Q19, R40
