File: hw/PIB/monarch_payload_interface_board_rev2/power supply.kicad_sch (KiCad schematic)
At the start: 26 parts, among them U14 WSK06121L000FEA, U4 TPS61088QRHLRQ1

Commit message: MCU Power Pins Fix
Other:
- moved on the sheet: C1, C10, C2, C3, C4, C5, C51, C52, C53, C54, C6, C7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

Commit message: Connector Additions
Other:
- note added: "TPS61088-Q1 10-A Fully-Integrated Synchronous Boost Converter"
Changed lines of the file:
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@@
 	)
 	(rectangle
-		(start 45.72 51.054)
-		(end 73.66 63.5)
+		(start 24.13 152.654)
+		(end 52.07 165.1)
 		(stroke
 			(width 0)
@@
 		)
 	)
+	(text "TPS61088-Q1 10-A Fully-Integrated Synchronous Boost Converter\n\n"
+		(exclude_from_sim no)
+		(at 84.582 44.704 0)
+		(effects
+			(font
+				(size 2.286 2.286)
+			)
+		)
+	)
 	(junction
 		(at 231.14 64.77)
@@
 	(wire
 		(pts
-			(xy 54.61 53.34) (xy 62.23 53.34)
+			(xy 33.02 154.94) (xy 40.64 154.94)
 		)
 		(stroke
@@
 	(wire
 		(pts
-			(xy 54.61 60.96) (xy 62.23 60.96)
+			(xy 33.02 162.56) (xy 40.64 162.56)
 		)
 		(stroke
@@
 	(wire
 		(pts
-			(xy 54.61 57.15) (xy 62.23 57.15)
+			(xy 33.02 158.75) (xy 40.64 158.75)
 		)
 		(stroke
@@
 	(hierarchical_label "GND"
 		(shape input)
-		(at 54.61 53.34 180)
+		(at 33.02 154.94 180)
 		(effects
 			(font
@@
 	(hierarchical_label "+12VB"
 		(shape input)
-		(at 54.61 60.96 180)
+		(at 33.02 162.56 180)
 		(effects
 			(font
@@
 	(hierarchical_label "VBAT"
 		(shape input)
-		(at 54.61 57.15 180)
+		(at 33.02 158.75 180)
 		(effects
 			(font
@@
 	(symbol
 		(lib_id "power:VBUS")
-		(at 62.23 57.15 270)
+		(at 40.64 158.75 270)
 		(unit 1)
 		(body_style 1)
@@
 		(fields_autoplaced yes)
 		(property "Reference" "#PWR0105"
-			(at 58.42 57.15 0)
+			(at 36.83 158.75 0)
 			(hide yes)
 			(show_name no)
@@
 		)
 		(property "Value" "VBAT"
-			(at 66.04 57.1499 90)
+			(at 44.45 158.7499 90)
 			(show_name no)
 			(do_not_autoplace no)
@@
 		)
 		(property "Footprint" ""
-			(at 62.23 57.15 0)
+			(at 40.64 158.75 0)
 			(hide yes)
 			(show_name no)
@@
 		)
 		(property "Datasheet" ""
-			(at 62.23 57.15 0)
+			(at 40.64 158.75 0)
 			(hide yes)
 			(show_name no)
@@
 		)
 		(property "Description" "Power symbol creates a global label with name \"VBUS\""
-			(at 62.23 57.15 0)
+			(at 40.64 158.75 0)
 			(hide yes)
 			(show_name no)
@@
 	(symbol
 		(lib_id "power:GND")
-		(at 62.23 53.34 90)
+		(at 40.64 154.94 90)
 		(unit 1)
 		(body_style 1)
@@
 		(fields_autoplaced yes)
 		(property "Reference" "#PWR05"
-			(at 68.58 53.34 0)
+			(at 46.99 154.94 0)
 			(hide yes)
 			(show_name no)
@@
 		)
 		(property "Value" "GND"
-			(at 66.04 53.3399 90)
+			(at 44.45 154.9399 90)
 			(show_name no)
 			(do_not_autoplace no)
@@
 		)
 		(property "Footprint" ""
-			(at 62.23 53.34 0)
+			(at 40.64 154.94 0)
 			(hide yes)
 			(show_name no)
@@
 		)
 		(property "Datasheet" ""
-			(at 62.23 53.34 0)
+			(at 40.64 154.94 0)
 			(hide yes)
 			(show_name no)
@@
 		)
 		(property "Description" "Power symbol creates a global label with name \"GND\" , ground"
-			(at 62.23 53.34 0)
+			(at 40.64 154.94 0)
 			(hide yes)
 			(show_name no)
@@
 	(symbol
 		(lib_id "power:VBUS")
-		(at 62.23 60.96 270)
+		(at 40.64 162.56 270)
 		(unit 1)
 		(body_style 1)
@@
 		(fields_autoplaced yes)
 		(property "Reference" "#PWR0107"
-			(at 58.42 60.96 0)
+			(at 36.83 162.56 0)
 			(hide yes)
 			(show_name no)
@@
 		)
 		(property "Value" "+12VB"
-			(at 66.04 60.9599 90)
+			(at 44.45 162.5599 90)
 			(show_name no)
 			(do_not_autoplace no)
@@
 		)
 		(property "Footprint" ""
-			(at 62.23 60.96 0)
+			(at 40.64 162.56 0)
 			(hide yes)
 			(show_name no)
@@
 		)
 		(property "Datasheet" ""
-			(at 62.23 60.96 0)
+			(at 40.64 162.56 0)
 			(hide yes)
 			(show_name no)
@@
 		)
 		(property "Description" "Power symbol creates a global label with name \"VBUS\""
-			(at 62.23 60.96 0)
+			(at 40.64 162.56 0)
 			(hide yes)
 			(show_name no)
