File: hw/PIB/monarch_payload_interface_board_rev2/power supply.kicad_sch (KiCad schematic)
At the start: 26 parts, among them U14 WSK06121L000FEA, U4 TPS61088QRHLRQ1

Commit message: Schematic Clean Up + New Micro-Lock Plus Connectors
Parts:
- U14: footprint WSK:SMT_121L000FEA_VIS -> SMT_121L000FEA_VIS
- U4: footprint tps6:RHL0020A -> RHL0020A
Changed lines of the file:
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@@
 			)
 		)
-		(property "Footprint" "tps6:RHL0020A"
+		(property "Footprint" "RHL0020A"
 			(at 120.65 102.87 0)
 			(hide yes)
@@
 			)
 		)
-		(property "Footprint" "WSK:SMT_121L000FEA_VIS"
+		(property "Footprint" "SMT_121L000FEA_VIS"
 			(at 242.57 64.77 0)
 			(hide yes)

Commit message: Schematic Updates Finished -> AD7124 Voltage Reading Fix + Connector Linkage Issue Fix
Connections:
- net 12VB_VA renamed 12VB_VA+
- net 12VB_VB renamed 12VB_VB+
Other:
- moved on the sheet: R46
Changed lines of the file:
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@@
 	(paper "A4")
 	(rectangle
-		(start 24.13 39.37)
-		(end 273.05 151.13)
+		(start 19.05 39.37)
+		(end 280.67 151.13)
 		(stroke
 			(width 0)
@@
 	)
 	(junction
-		(at 231.14 64.77)
-		(diameter 0)
-		(color 0 0 0 0)
-	)
-	(junction
 		(at 158.75 68.58)
 		(diameter 0)
@@
 	)
 	(junction
+		(at 255.27 64.77)
+		(diameter 0)
+		(color 0 0 0 0)
+	)
+	(junction
+		(at 220.98 64.77)
+		(diameter 0)
+		(color 0 0 0 0)
+	)
+	(junction
 		(at 73.66 100.33)
 		(diameter 0)
@@
 	)
 	(junction
-		(at 251.46 64.77)
+		(at 228.6 64.77)
 		(diameter 0)
 		(color 0 0 0 0)
@@
 	)
 	(junction
+		(at 262.89 64.77)
+		(diameter 0)
+		(color 0 0 0 0)
+	)
+	(junction
 		(at 59.69 67.31)
 		(diameter 0)
@@
 	(wire
 		(pts
+			(xy 262.89 54.61) (xy 262.89 64.77)
+		)
+		(stroke
+			(width 0)
+			(type default)
+		)
+	)
+	(wire
+		(pts
 			(xy 138.43 85.09) (xy 140.97 85.09)
 		)
@@
 	(wire
 		(pts
-			(xy 251.46 64.77) (xy 251.46 54.61)
+			(xy 264.16 64.77) (xy 262.89 64.77)
 		)
 		(stroke
@@
 	(wire
 		(pts
-			(xy 264.16 64.77) (xy 260.35 64.77)
+			(xy 95.25 68.58) (xy 109.22 68.58)
 		)
 		(stroke
@@
 	(wire
 		(pts
-			(xy 95.25 68.58) (xy 109.22 68.58)
+			(xy 220.98 64.77) (xy 222.25 64.77)
 		)
 		(stroke
@@
 	(wire
 		(pts
-			(xy 227.33 107.95) (xy 227.33 111.76)
+			(xy 228.6 64.77) (xy 233.68 64.77)
 		)
 		(stroke
@@
 	(wire
 		(pts
-			(xy 231.14 64.77) (xy 231.14 54.61)
+			(xy 227.33 107.95) (xy 227.33 111.76)
 		)
 		(stroke
@@
 	(wire
 		(pts
-			(xy 208.28 107.95) (xy 208.28 111.76)
+			(xy 228.6 64.77) (xy 228.6 54.61)
 		)
 		(stroke
@@
 	(wire
 		(pts
-			(xy 238.76 64.77) (xy 240.03 64.77)
+			(xy 208.28 107.95) (xy 208.28 111.76)
 		)
 		(stroke
@@
 	(wire
 		(pts
-			(xy 231.14 64.77) (xy 233.68 64.77)
+			(xy 238.76 64.77) (xy 240.03 64.77)
 		)
 		(stroke
@@
 	(wire
 		(pts
-			(xy 227.33 64.77) (xy 231.14 64.77)
+			(xy 227.33 64.77) (xy 228.6 64.77)
 		)
 		(stroke
@@
 	(wire
 		(pts
+			(xy 262.89 64.77) (xy 261.62 64.77)
+		)
+		(stroke
+			(width 0)
+			(type default)
+		)
+	)
+	(wire
+		(pts
 			(xy 33.02 162.56) (xy 40.64 162.56)
 		)
@@
 	(wire
 		(pts
-			(xy 251.46 64.77) (xy 248.92 64.77)
+			(xy 248.92 64.77) (xy 255.27 64.77)
 		)
 		(stroke
@@
 	(wire
 		(pts
-			(xy 218.44 64.77) (xy 222.25 64.77)
+			(xy 218.44 64.77) (xy 220.98 64.77)
 		)
 		(stroke
@@
 	(wire
 		(pts
-			(xy 255.27 64.77) (xy 251.46 64.77)
+			(xy 220.98 54.61) (xy 220.98 64.77)
 		)
 		(stroke
@@
 	(wire
 		(pts
+			(xy 256.54 64.77) (xy 255.27 64.77)
+		)
+		(stroke
+			(width 0)
+			(type default)
+		)
+	)
+	(wire
+		(pts
 			(xy 57.15 67.31) (xy 59.69 67.31)
 		)
@@
 		)
 	)
-	(global_label "12VB_VB"
-		(shape output)
-		(at 231.14 54.61 0)
+	(wire
+		(pts
+			(xy 255.27 54.61) (xy 255.27 64.77)
+		)
+		(stroke
+			(width 0)
+			(type default)
+		)
+	)
+	(global_label "12VB_VB-"
+		(shape input)
+		(at 220.98 54.61 180)
+		(fields_autoplaced yes)
+		(effects
+			(font
+				(size 1.27 1.27)
+			)
+			(justify right)
+		)
+		(property "Intersheetrefs" "${INTERSHEET_REFS}"
+			(at 208.9728 54.61 0)
+			(hide yes)
+			(show_name no)
+			(do_not_autoplace no)
+			(effects
+				(font
+					(size 1.27 1.27)
+				)
+				(justify right)
+			)
+		)
+	)
+	(global_label "12VB_VB+"
+		(shape input)
+		(at 228.6 54.61 0)
 		(fields_autoplaced yes)
 		(effects
@@
 		)
 		(property "Intersheetrefs" "${INTERSHEET_REFS}"
-			(at 241.5748 54.61 0)
+			(at 240.6072 54.61 0)
 			(hide yes)
 			(show_name no)
@@
 		)
 	)
-	(global_label "12VB_VA"
-		(shape output)
-		(at 251.46 54.61 0)
+	(global_label "12VB_VA-"
+		(shape input)
+		(at 262.89 54.61 0)
 		(fields_autoplaced yes)
 		(effects
@@
 		)
 		(property "Intersheetrefs" "${INTERSHEET_REFS}"
-			(at 261.7134 54.61 0)
+			(at 274.7158 54.61 0)
 			(hide yes)
 			(show_name no)
@@
 		)
 	)
+	(global_label "12VB_VA+"
+		(shape input)
+		(at 255.27 54.61 180)
+		(fields_autoplaced yes)
+		(effects
+			(font
+				(size 1.27 1.27)
+			)
+			(justify right)
+		)
+		(property "Intersheetrefs" "${INTERSHEET_REFS}"
+			(at 243.4442 54.61 0)
+			(hide yes)
+			(show_name no)
+			(do_not_autoplace no)
+			(effects
+				(font
+					(size 1.27 1.27)
+				)
+				(justify right)
+			)
+		)
+	)
 	(hierarchical_label "GND"
 		(shape input)
@@
 	(symbol
 		(lib_id "Device:R_Small")
-		(at 257.81 64.77 270)
+		(at 259.08 64.77 270)
 		(unit 1)
 		(body_style 1)
@@
 		(dnp no)
 		(property "Reference" "R46"
-			(at 257.81 60.706 90)
+			(at 259.08 60.706 90)
 			(show_name no)
 			(do_not_autoplace no)
@@
 		)
 		(property "Value" "100k"
-			(at 258.064 62.738 90)
+			(at 259.334 62.738 90)
 			(show_name no)
 			(do_not_autoplace no)
@@
 		)
 		(property "Footprint" "Resistor_SMD:R_0603_1608Metric"
-			(at 257.81 64.77 0)
+			(at 259.08 64.77 0)
 			(hide yes)
 			(show_name no)
@@
 		)
 		(property "Datasheet" ""
-			(at 257.81 64.77 0)
+			(at 259.08 64.77 0)
 			(hide yes)
 			(show_name no)
@@
 		)
 		(property "Description" "Resistor, small symbol"
-			(at 257.81 64.77 0)
+			(at 259.08 64.77 0)
 			(hide yes)
 			(show_name no)

Commit message: Footprint Selected
Parts:
- U14: footprint SMT_121L000FEA_VIS -> WSK:SMT_121L000FEA_VIS
- U4: footprint RHL0020A -> tps6:RHL0020A
Changed lines of the file:
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@@
 			)
 		)
-		(property "Footprint" "RHL0020A"
+		(property "Footprint" "tps6:RHL0020A"
 			(at 120.65 102.87 0)
 			(hide yes)
@@
 			)
 		)
-		(property "Footprint" "SMT_121L000FEA_VIS"
+		(property "Footprint" "WSK:SMT_121L000FEA_VIS"
 			(at 242.57 64.77 0)
 			(hide yes)
