File: hw/PIB/monarch_payload_interface_board_rev2/MCU.kicad_sch (KiCad schematic)
At the start: 30 parts, among them J16 20021121-00008C4LF, J17 Conn_02x04_Counter_Clockwise, SW1 SW_BOOT, SW2 SW_RESET, U2 STM32L4A6VGTx

Commit message: Schematic Clean Up + New Micro-Lock Plus Connectors
Parts:
- removed J16: 20021121-00008C4LF, 20021121:AMPHENOL_20021121-00008C4LF, symbol 20021121:20021121-00008C4LF
Changed lines of the file:
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@@
-	)
-	(symbol
-		(lib_id "20021121:20021121-00008C4LF")
-		(at 317.5 25.4 0)
-		(unit 1)
-		(body_style 1)
-		(exclude_from_sim no)
-		(in_bom yes)
-		(on_board yes)
-		(in_pos_files yes)
-		(dnp no)
-		(fields_autoplaced yes)
-		(property "Reference" "J16"
-			(at 317.5 12.7 0)
-			(show_name no)
-			(do_not_autoplace no)
-			(effects
-				(font
-					(size 1.27 1.27)
-				)
-			)
-		)
-		(property "Value" "20021121-00008C4LF"
-			(at 317.5 15.24 0)
-			(show_name no)
-			(do_not_autoplace no)
-			(effects
-				(font
-					(size 1.27 1.27)
-				)
-			)
-		)
-		(property "Footprint" "20021121:AMPHENOL_20021121-00008C4LF"
-			(at 317.5 25.4 0)
-			(hide yes)
-			(show_name no)
-			(do_not_autoplace no)
-			(effects
-				(font
-					(size 1.27 1.27)
-				)
-				(justify bottom)
-			)
-		)
-		(property "Datasheet" ""
-			(at 317.5 25.4 0)
-			(hide yes)
-			(show_name no)
-			(do_not_autoplace no)
-			(effects
-				(font
-					(size 1.27 1.27)
-				)
-			)
-		)
-		(property "Description" ""
-			(at 317.5 25.4 0)
-			(hide yes)
-			(show_name no)
-			(do_not_autoplace no)
-			(effects
-				(font
-					(size 1.27 1.27)
-				)
-			)
-		)
-		(property "DigiKey_Part_Number" "609-3694-1-ND"
-			(at 317.5 25.4 0)
-			(hide yes)
-			(show_name no)
-			(do_not_autoplace no)
-			(effects
-				(font
-					(size 1.27 1.27)
-				)
-				(justify bottom)
-			)
-		)
-		(property "SnapEDA_Link" "https://www.snapeda.com/parts/20021121-00008C4LF/Amphenol/view-part/?ref=snap"
-			(at 317.5 25.4 0)
-			(hide yes)
-			(show_name no)
-			(do_not_autoplace no)
-			(effects
-				(font
-					(size 1.27 1.27)
-				)
-				(justify bottom)
-			)
-		)
-		(property "Description_1" "Conn Rect Header Unshrouded 1.27x1.27 mm 8 Pos SMT Minitek127 BtoB | Amphenol FCI (Amphenol CS) 20021121-00008C4LF"
-			(at 317.5 25.4 0)
-			(hide yes)
-			(show_name no)
-			(do_not_autoplace no)
-			(effects
-				(font
-					(size 1.27 1.27)
-				)
-				(justify bottom)
-			)
-		)
-		(property "Package" "None"
-			(at 317.5 25.4 0)
-			(hide yes)
-			(show_name no)
-			(do_not_autoplace no)
-			(effects
-				(font
-					(size 1.27 1.27)
-				)
-				(justify bottom)
-			)
-		)
-		(property "Check_prices" "https://www.snapeda.com/parts/20021121-00008C4LF/Amphenol/view-part/?ref=eda"
-			(at 317.5 25.4 0)
-			(hide yes)
-			(show_name no)
-			(do_not_autoplace no)
-			(effects
-				(font
-					(size 1.27 1.27)
-				)
-				(justify bottom)
-			)
-		)
-		(property "MF" "Amphenol ICC"
-			(at 317.5 25.4 0)
-			(hide yes)
-			(show_name no)
-			(do_not_autoplace no)
-			(effects
-				(font
-					(size 1.27 1.27)
-				)
-				(justify bottom)
-			)
-		)
-		(property "MP" "20021121-00008C4LF"
-			(at 317.5 25.4 0)
-			(hide yes)
-			(show_name no)
-			(do_not_autoplace no)
-			(effects
-				(font
-					(size 1.27 1.27)
-				)
-				(justify bottom)
-			)
-		)
-		(property "MANUFACTURER" "AMPHENOL"
-			(at 317.5 25.4 0)
-			(hide yes)
-			(show_name no)
-			(do_not_autoplace no)
-			(effects
-				(font
-					(size 1.27 1.27)
-				)
-				(justify bottom)
-			)
-		)
-		(pin "2"
-		)
-		(pin "5"
-		)
-		(pin "4"
-		)
-		(pin "3"
-		)
-		(pin "7"
-		)
-		(pin "8"
-		)
-		(pin "6"
-		)
-		(pin "1"
-		)
-		(instances
-			(project "monarch_payload_interface_board_rev2"
-				(path "/bf7ee58d-ac53-49d1-a6b2-96a87d67b737/15dbdbb2-29d8-485f-9d04-213689f007b4"
-					(reference "J16")
-					(unit 1)
-				)
-			)
-		)
 	)
 	(symbol

Commit message: AD7124 Fixes
Parts:
- R56, R58: value 1000 -> 125
Changed lines of the file:
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@@
 			)
 		)
-		(property "Value" "1000"
+		(property "Value" "125"
 			(at 205.74 96.52 90)
 			(show_name no)
@@
 			)
 		)
-		(property "Value" "1000"
+		(property "Value" "125"
 			(at 205.74 84.328 90)
 			(show_name no)

Commit message: AD7124 fixes
Parts:
- J17: footprint (none) -> Connector_PinHeader_2.54mm:PinHeader_2x04_P2.54mm_Vertical
Changed lines of the file:
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@@
 			)
 		)
-		(property "Footprint" ""
+		(property "Footprint" "Connector_PinHeader_2.54mm:PinHeader_2x04_P2.54mm_Vertical"
 			(at 210.82 34.29 0)
 			(hide yes)

Commit message: Schematic Updates Finished -> AD7124 Voltage Reading Fix + Connector Linkage Issue Fix
Parts:
- added D5, D6, D7: LED, LED_SMD:LED_0603_1608Metric, symbol Device:LED
- added R59: 125, Resistor_SMD:R_0603_1608Metric, symbol Device:R_Small
- added R60, R64: 1000, Resistor_SMD:R_0603_1608Metric, symbol Device:R_Small
Connections:
- net +3V3: now also R59.2
- net GND: now also D5.1 (K), D6.1 (K), D7.1 (K)
- net *SYNC: now reaches U2.91 (PB5)
- new net: D7.2 (A), R64.1
- new net: D5.2 (A), R59.1
- new net: D6.2 (A), R60.1
- new net +12VA: R64.2
- new net +12VB: R60.2
Other:
- note added: "Power LEDS"
