File: hw/PIB/monarch_payload_interface_board_rev2/MCU.kicad_sch (KiCad schematic)
At the start: 35 parts, among them J17 Conn_02x04_Counter_Clockwise, SW1 SW_BOOT, SW2 SW_RESET, U2 STM32L4A6VGTx

Commit message: Footprint Selected
Parts:
- SW1, SW2: footprint (none) -> Connector_PinHeader_1.00mm:PinHeader_1x02_P1.00mm_Vertical
Changed lines of the file:
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@@
 			)
 		)
-		(property "Footprint" ""
+		(property "Footprint" "Connector_PinHeader_1.00mm:PinHeader_1x02_P1.00mm_Vertical"
 			(at 66.04 81.28 0)
 			(hide yes)
@@
 			)
 		)
-		(property "Footprint" ""
+		(property "Footprint" "Connector_PinHeader_1.00mm:PinHeader_1x02_P1.00mm_Vertical"
 			(at 64.77 43.18 0)
 			(hide yes)

Commit message: Initial Routing Work + Placement
Connections:
- no-connect marks 1 -> 0
Changed lines of the file:
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@@
 		(color 0 0 0 0)
-	)
-	(no_connect
-		(at 139.7 30.48)
 	)
 	(wire

Commit message: Great progress almost done
Connections:
- net Valve6: now also U2.4 (PE5); no longer U2.40 (PE9)
- no-connect marks 0 -> 35
Changed lines of the file:
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@@
 		(color 0 0 0 0)
 	)
+	(no_connect
+		(at 76.2 104.14)
+	)
+	(no_connect
+		(at 76.2 106.68)
+	)
+	(no_connect
+		(at 76.2 137.16)
+	)
+	(no_connect
+		(at 76.2 109.22)
+	)
+	(no_connect
+		(at 121.92 114.3)
+	)
+	(no_connect
+		(at 121.92 116.84)
+	)
+	(no_connect
+		(at 76.2 93.98)
+	)
+	(no_connect
+		(at 76.2 149.86)
+	)
+	(no_connect
+		(at 76.2 154.94)
+	)
+	(no_connect
+		(at 121.92 175.26)
+	)
+	(no_connect
+		(at 121.92 101.6)
+	)
+	(no_connect
+		(at 76.2 71.12)
+	)
+	(no_connect
+		(at 76.2 139.7)
+	)
+	(no_connect
+		(at 121.92 104.14)
+	)
+	(no_connect
+		(at 76.2 96.52)
+	)
+	(no_connect
+		(at 76.2 101.6)
+	)
+	(no_connect
+		(at 121.92 60.96)
+	)
+	(no_connect
+		(at 76.2 99.06)
+	)
+	(no_connect
+		(at 121.92 144.78)
+	)
+	(no_connect
+		(at 76.2 134.62)
+	)
+	(no_connect
+		(at 76.2 160.02)
+	)
+	(no_connect
+		(at 121.92 119.38)
+	)
+	(no_connect
+		(at 121.92 86.36)
+	)
+	(no_connect
+		(at 76.2 152.4)
+	)
+	(no_connect
+		(at 76.2 157.48)
+	)
+	(no_connect
+		(at 121.92 78.74)
+	)
+	(no_connect
+		(at 121.92 63.5)
+	)
+	(no_connect
+		(at 121.92 142.24)
+	)
+	(no_connect
+		(at 121.92 180.34)
+	)
+	(no_connect
+		(at 121.92 99.06)
+	)
+	(no_connect
+		(at 76.2 147.32)
+	)
+	(no_connect
+		(at 76.2 73.66)
+	)
+	(no_connect
+		(at 121.92 177.8)
+	)
+	(no_connect
+		(at 121.92 149.86)
+	)
+	(no_connect
+		(at 121.92 147.32)
+	)
 	(wire
 		(pts
@@
 	(wire
 		(pts
-			(xy 73.66 101.6) (xy 76.2 101.6)
-		)
-		(stroke
-			(width 0)
-			(type default)
-		)
-	)
-	(wire
-		(pts
 			(xy 73.66 132.08) (xy 76.2 132.08)
 		)
@@
 	(wire
 		(pts
-			(xy 73.66 93.98) (xy 76.2 93.98)
-		)
-		(stroke
-			(width 0)
-			(type default)
-		)
-	)
-	(wire
-		(pts
 			(xy 76.2 121.92) (xy 73.66 121.92)
 		)
@@
 		(pts
 			(xy 93.98 24.13) (xy 96.52 24.13)
+		)
+		(stroke
+			(width 0)
+			(type default)
+		)
+	)
+	(wire
+		(pts
+			(xy 73.66 91.44) (xy 76.2 91.44)
 		)
 		(stroke
@@
 	(hierarchical_label "Valve6"
 		(shape output)
-		(at 73.66 101.6 180)
+		(at 73.66 91.44 180)
 		(effects
 			(font
@@
 	)
 	(hierarchical_label "GREEN_LED"
-		(shape input)
+		(shape output)
 		(at 199.39 93.98 180)
 		(effects
@@
 	)
 	(hierarchical_label "BLUE_LED"
-		(shape input)
+		(shape output)
 		(at 71.12 111.76 180)
 		(effects
@@
 	)
 	(hierarchical_label "RED_LED"
-		(shape input)
+		(shape output)
 		(at 199.39 69.85 180)
 		(effects
@@
 	)
 	(hierarchical_label "BLUE_LED"
-		(shape input)
+		(shape output)
 		(at 199.39 81.28 180)
 		(effects
@@
 	)
 	(hierarchical_label "RED_LED"
-		(shape input)
+		(shape output)
 		(at 71.12 116.84 180)
 		(effects
@@
 	)
 	(hierarchical_label "GREEN_LED"
-		(shape input)
+		(shape output)
 		(at 71.12 114.3 180)
 		(effects

Commit message: FINAL REVIEW DONE + A lot of fixes. DRC PASSED
Changed lines of the file:
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@@
 	)
 	(hierarchical_label "GREEN_LED"
-		(shape output)
+		(shape input)
 		(at 199.39 93.98 180)
 		(effects
@@
 	)
 	(hierarchical_label "BLUE_LED"
-		(shape output)
+		(shape input)
 		(at 71.12 111.76 180)
 		(effects
@@
 	)
 	(hierarchical_label "RED_LED"
-		(shape output)
+		(shape input)
 		(at 199.39 69.85 180)
 		(effects
@@
 	)
 	(hierarchical_label "BLUE_LED"
-		(shape output)
+		(shape input)
 		(at 199.39 81.28 180)
 		(effects
@@
 	)
 	(hierarchical_label "RED_LED"
-		(shape output)
+		(shape input)
 		(at 71.12 116.84 180)
 		(effects
@@
 	)
 	(hierarchical_label "GREEN_LED"
-		(shape output)
+		(shape input)
 		(at 71.12 114.3 180)
 		(effects

Commit message: Schematic Unconnected Fix
Connections:
- no-connect marks 35 -> 34
Changed lines of the file:
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@@
-	)
-	(no_connect
-		(at 76.2 73.66)
 	)
 	(no_connect
@@
 	)
 	(hierarchical_label "GREEN_LED"
-		(shape input)
+		(shape output)
 		(at 199.39 93.98 180)
 		(effects
@@
 	)
 	(hierarchical_label "BLUE_LED"
-		(shape input)
+		(shape output)
 		(at 71.12 111.76 180)
 		(effects
@@
 	)
 	(hierarchical_label "RED_LED"
-		(shape input)
+		(shape output)
 		(at 199.39 69.85 180)
 		(effects
@@
 	)
 	(hierarchical_label "BLUE_LED"
-		(shape input)
+		(shape output)
 		(at 199.39 81.28 180)
 		(effects
@@
 	)
 	(hierarchical_label "RED_LED"
-		(shape input)
+		(shape output)
 		(at 71.12 116.84 180)
 		(effects
@@
 	)
 	(hierarchical_label "GREEN_LED"
-		(shape input)
+		(shape output)
 		(at 71.12 114.3 180)
 		(effects
