File: hw/PIB/monarch_payload_interface_board_rev2/circuit-diagram.kicad_sch (KiCad schematic)
At the start: 204 parts, among them J10 2200980671, J11 Conn_01x04, J12 Conn_01x05, J26 Conn_02x04_Counter_Clockwise, J27 2200980271, J28 2200980471, J29 2200980671, J30 2200980671, J31 2200980671, J32 2200980671, J33 Conn_01x05, J34 2200980671, J35 2200980671, J36 2200980471, J37 2200980471, J38 2200980471, J39 Conn_01x06, J40 2200980671, J7 2200980271, J9 2200980671, Q20 FZT600TA, Q21 FZT600TA, Q22 FZT600TA, Q23 FZT600TA, Q24 FZT600TA, Q25 FZT600TA, Q26 FZT600TA, Q27 FZT600TA, Q28 FZT600TA, Q29 FZT600TA, Q30 FZT600TA, Q31 FZT600TA, Q32 FZT600TA, Q33 FZT600TA, Q34 FZT600TA, Q35 FZT600TA, Q36 FZT600TA, Q37 FZT600TA, Q38 FZT600TA, SW3 SW_BOOT, SW4 SW_RESET, U15 AD7124-8BCPZ-RL, U16 Payload, U17 WSK06121L000FEA, U18 WSK06121L000FEA, U19 WSK06121L000FEA, U20 STM32L4A6VGTx, U21 TPS61088QRHLRQ1, U22 WSK06121L000FEA, U23 MAX31856MUD_T, U24 MAX31856MUD_T, U25 MAX31856MUD_T, U26 MAX31856MUD_T, U27 MAX31856MUD_T

Commit message: Circuit Diagram Progress Almost Done
Parts:
- added C145, C146, C147, C148, C149, C150, C152, C153, C154, C155: 0.1u, Capacitor_SMD:C_0603_1608Metric, symbol Device:C_Small
- added C151, C156: 1u, Capacitor_SMD:C_0603_1608Metric, symbol Device:C_Small
- added R118, R119, R120, R121, R122, R123, R125, R126: 125, Resistor_SMD:R_0603_1608Metric, symbol Device:R_Small
- added R124: 10k, Resistor_SMD:R_0603_1608Metric, symbol Device:R_Small
- added U28: AD7124-8BCPZ-RL, AD7124:CP-32-12_ADI, symbol AD7124:AD7124-8BCPZ-RL
Connections:
- net NRST is gone; now on an unnamed net: U16.31
- net P0+ is gone; now on net +12VA: J34.1
- net P1+ is gone; now on net +12VA: J34.3
- net P2+ is gone; now on net +12VA: J34.5
- net P3+ is gone; now on net +12VA: J35.1
- net P4+ is gone; now on net +12VA: J35.3
- net P5+ is gone; now on net +12VA: J35.5
- net P6+ is gone; now on net +12VA: J36.1
- net P7+ is gone; now on net +12VA: J36.3
- net +12VA: no longer CR21.1
- net +3V3: now also C146.2, C152.1, C154.2, C156.2, R124.2, U28.2 (IOVDD), U28.26 (AVDD)
- net ADC: no longer U15.32 (*CS), U20.29 (PA4)
- net GND: now also C145.2, C146.1, C147.2, C148.1, C148.2, C149.2, C150.1, C151.1, C151.2, C152.2, C153.1, C153.2, C154.1, C155.1, C156.1, R118.1, R119.1, R120.1, R121.1, R122.1, R123.1, R125.1, R126.1, U28.11 (AIN7/IOUT/VBIAS), U28.13 (REFIN1(-)), U28.15 (AIN9/IOUT/VBIAS), U28.17 (AIN11/IOUT/VBIAS), U28.19 (AIN13/IOUT/VBIAS), U28.21 (AIN15/IOUT/VBIAS/REFIN2(-)), U28.23 (AVSS), U28.3 (DGND), U28.33 (EP), U28.5 (AIN1/IOUT/VBIAS), U28.7 (AIN3/IOUT/VBIAS/P2), U28.9 (AIN5/IOUT/VBIAS/P4)
- net PT: now also U28.32 (*CS)
- net SPI1_MISO: no longer U15.28 (DOUT/*RDY), U20.31 (PA6)
- net SPI1_MOSI: no longer U15.29 (DIN), U20.32 (PA7)
- net SPI1_SCK: no longer U15.30 (SCLK), U20.30 (PA5)
- net SPI2_MISO: now also U28.28 (DOUT/*RDY); no longer U20.84 (PD3), U23.11 (SDO), U24.11 (SDO), U25.11 (SDO), U26.11 (SDO), U27.11 (SDO)
- net SPI2_MOSI: now also U28.29 (DIN); no longer U20.85 (PD4), U23.12 (SDI), U24.12 (SDI), U25.12 (SDI), U26.12 (SDI), U27.12 (SDI)
- net SPI2_SCK: now also U28.30 (SCLK); no longer U20.82 (PD1), U23.10 (SCK), U24.10 (SCK), U25.10 (SCK), U26.10 (SCK), U27.10 (SCK)
- net T1: no longer U20.96 (PB9), U24.9 (~{CS})
- net T2: no longer U20.2 (PE3), U26.9 (~{CS})
- net T3: no longer U20.97 (PE0), U23.9 (~{CS})
- net T4: no longer U20.1 (PE2), U25.9 (~{CS})
- net T5: no longer U20.98 (PE1), U27.9 (~{CS})
- net USART3_RX: no longer U20.34 (PC5)
- net USART3_TX: no longer U20.33 (PC4)
- net P0- renamed P0REF+
- net P0REF+: now also R118.2, U28.4 (AIN0/IOUT/VBIAS)
- net P1- renamed P1REF+
- net P1REF+: now also R120.2, U28.6 (AIN2/IOUT/VBIAS/P1)
- net P2- renamed P2REF+
- net P2REF+: now also R122.2, U28.8 (AIN4/IOUT/VBIAS/P3)
- net P3- renamed P3REF+
- net P3REF+: now also R125.2, U28.10 (AIN6/IOUT/VBIAS)
- net P4- renamed P4REF+
- net P4REF+: now also R119.2, U28.14 (AIN8/IOUT/VBIAS)
- net P5- renamed P5REF+
- net P5REF+: now also R121.2, U28.16 (AIN10/IOUT/VBIAS)
- net P6- renamed P6REF+
- net P6REF+: now also R123.2, U28.18 (AIN12/IOUT/VBIAS)
- net P7- renamed P7REF+
- net P7REF+: now also R126.2, U28.20 (AIN14/IOUT/VBIAS/REFIN2(+))
- net UART_RX: no longer names the net of U16.33
- net UART_RX: now also U20.34 (PC5)
- net UART_TX: no longer names the net of U16.35
- net UART_TX: now also U20.33 (PC4)
- net Valve10: no longer names the net of R104.2, R106.1, U20.65 (PC8)
- net Valve11: no longer names the net of R89.1, U20.66 (PC9)
- net Valve12: no longer names the net of R95.1, U20.67 (PA8)
- net Valve13: no longer names the net of R99.1, U20.78 (PC10)
- net Valve14: no longer names the net of R103.1, U20.79 (PC11)
- net Valve15: no longer names the net of R107.1, U20.83 (PD2)
- net Valve16: no longer names the net of R90.1, U20.80 (PC12)
- net Valve17: no longer names the net of R92.2, R96.1, U20.81 (PD0)
- net Valve18: no longer names the net of R100.1, U20.70 (PA11)
- net Valve6: no longer names the net of R88.1, U20.40 (PE9)
- net Valve7: no longer names the net of R94.1, U20.55 (PD8)
- net Valve8: no longer names the net of R98.1, U20.56 (PD9)
- net Valve9: no longer names the net of R102.1, U20.64 (PC7)
- new net: U20.82 (PD1), U23.10 (SCK), U24.10 (SCK), U25.10 (SCK), U26.10 (SCK), U27.10 (SCK)
- new net: U20.84 (PD3), U23.11 (SDO), U24.11 (SDO), U25.11 (SDO), U26.11 (SDO), U27.11 (SDO)
- new net: U20.85 (PD4), U23.12 (SDI), U24.12 (SDI), U25.12 (SDI), U26.12 (SDI), U27.12 (SDI)
- new net: U20.2 (PE3), U26.9 (~{CS})
- new net: C150.2, U28.1 (REGCAPD)
- new net: C145.1, C147.1, C149.1, U28.12 (REFIN1(+)), U28.22 (REFOUT)
- new net: U15.28 (DOUT/*RDY), U20.31 (PA6)
- new net: U15.29 (DIN), U20.32 (PA7)
- new net: U15.30 (SCLK), U20.30 (PA5)
- new net: U15.32 (*CS), U20.29 (PA4)
- new net: R124.1, U28.27 (*SYNC)
- new net: U20.1 (PE2), U25.9 (~{CS})
- new net: U20.96 (PB9), U24.9 (~{CS})
- new net: U20.97 (PE0), U23.9 (~{CS})
- new net: U20.98 (PE1), U27.9 (~{CS})
- new net: C155.2, U28.24 (REGCAPA)
- no-connect marks 88 -> 90
Other:
- note added: ".02 A (20mA max from pressure sensor) * 125 = 2.5 V (2.5 volt max reading from ad7124)"
- note added: "SPI2_MISO"
- note added: "SPI2_MOSI"
- note added: "SPI2_SCK"
- note added: "Solenoid Valves"
- note added: "T2"
- note added: "Temperature ADCs"
- note removed: "Vbat pin must be connected to VDD even if VBAT block (RTC.. etc ) is not used."
- note removed: "When the functions supplied by VDDA, VDDUSB or VDDIO2 are not used, these supplies should preferably be shorted to VDD."
- note removed: "filters out electrical noise"
- note removed: "nominally tied high but can always be pulled low by OBC"
- moved on the sheet: C100, C106, C107, C108, C109, C110, C111, C112, C113, C114, C115, C116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

Commit message: Work on Circuit Diagram
Parts:
- removed J35: 2200980671, Connector_Molex_Micro-Lock-Plus:Molex_Micro-Lock_2200980671_1x06_P1.25mm_Horizontal, symbol 5037630691:5037630691
- added J41: 2200980671, Connector_Molex_Micro-Lock-Plus:Molex_Micro-Lock_2200980671_1x06_P1.25mm_Horizontal, symbol 5037630691:5037630691
Connections:
- net USART3_RX is gone; now on an unnamed net: J11.3 (Pin_3)
- net USART3_TX is gone; now on an unnamed net: J11.4 (Pin_4)
- net *SYNC: no longer R78.1, U15.27 (*SYNC), U20.91 (PB5)
- net +12VA: now also J41.1, J41.3, J41.5
- net SPI2_MISO: no longer U28.28 (DOUT/*RDY)
- net SPI2_MOSI: no longer U28.29 (DIN)
- net SPI2_SCK: no longer U28.30 (SCLK)
- net UART_PPU_RX: no longer J11.2 (Pin_2)
- net UART_PPU_TX: no longer J11.1 (Pin_1)
- net at U20.82 (PD1), U23.10 (SCK), U24.10 (SCK)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: now also U28.30 (SCLK)
- net at U20.84 (PD3), U23.11 (SDO), U24.11 (SDO)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: now also U28.28 (DOUT/*RDY)
- net at U20.85 (PD4), U23.12 (SDI), U24.12 (SDI)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: now also U28.29 (DIN)
- net 12VA_VA+: no longer names the net of R67.2, R73.1, U15.18 (AIN12/IOUT/VBIAS)
- net 12VA_VB+: no longer names the net of R49.2, R72.1, U15.20 (AIN14/IOUT/VBIAS/REFIN2(+))
- net 12VB_VA+: no longer names the net of R115.1, R116.2, U15.6 (AIN2/IOUT/VBIAS/P1)
- net 12VB_VB+: no longer names the net of R113.2, R114.1, U15.4 (AIN0/IOUT/VBIAS)
- net 3V3_VA+: no longer names the net of R69.2, R75.1, U15.14 (AIN8/IOUT/VBIAS)
- net 3V3_VB+: no longer names the net of R68.2, R74.1, U15.16 (AIN10/IOUT/VBIAS)
- net EN: no longer names the net of U20.12 (PH0), U21.2 (EN)
- net Heater0-: no longer names the net of J37.2, Q38.2 (C_1), Q38.4 (C_2)
- net P0REF+: no longer names the net of J34.2, R118.2, U28.4 (AIN0/IOUT/VBIAS)
- net P1REF+: no longer names the net of J34.4, R120.2, U28.6 (AIN2/IOUT/VBIAS/P1)
- net P2REF+: no longer names the net of J34.6, R122.2, U28.8 (AIN4/IOUT/VBIAS/P3)
- net P3REF+: no longer names the net of R125.2, U28.10 (AIN6/IOUT/VBIAS)
- net P3REF+: now also J41.2
- net P4REF+: no longer names the net of R119.2, U28.14 (AIN8/IOUT/VBIAS)
- net P4REF+: now also J41.4
- net P5REF+: no longer names the net of R121.2, U28.16 (AIN10/IOUT/VBIAS)
- net P5REF+: now also J41.6
- net P6REF+: no longer names the net of J36.2, R123.2, U28.18 (AIN12/IOUT/VBIAS)
- net P7REF+: no longer names the net of J36.4, R126.2, U28.20 (AIN14/IOUT/VBIAS/REFIN2(+))
- net T0+: no longer names the net of C123.2, C124.1, J10.2, U24.4 (T+)
- net T0-: no longer names the net of C124.2, C125.1, J10.1, U24.2 (BIAS), U24.3 (T-)
- net T1+: no longer names the net of C133.2, C134.1, J10.4, U26.4 (T+)
- net T1-: no longer names the net of C134.2, C135.1, J10.3, U26.2 (BIAS), U26.3 (T-)
- net T2+: no longer names the net of C120.2, C121.1, J10.6, U23.4 (T+)
- net T2-: no longer names the net of C121.2, C122.1, J10.5, U23.2 (BIAS), U23.3 (T-)
- net T3+: no longer names the net of C130.2, C131.1, J28.2, U25.4 (T+)
- net T3-: no longer names the net of C131.2, C132.1, J28.1, U25.2 (BIAS), U25.3 (T-)
- net T4+: no longer names the net of C140.2, C141.1, J28.4, U27.4 (T+)
- net T4-: no longer names the net of C141.2, C142.1, J28.3, U27.2 (BIAS), U27.3 (T-)
- net UART4_RX: no longer names the net of U20.24 (PA1)
- net UART4_RX: now also J11.2 (Pin_2)
- net UART4_TX: no longer names the net of U20.23 (PA0)
- net UART4_TX: now also J11.1 (Pin_1)
- net VBAT_VA+: no longer names the net of R70.2, R76.1, U15.10 (AIN6/IOUT/VBIAS)
- net VBAT_VB+: no longer names the net of R71.2, R77.1, U15.8 (AIN4/IOUT/VBIAS/P3)
- net Valve1-: no longer names the net of CR19.2, J29.2, Q20.2 (C_1), Q20.4 (C_2)
- net Valve12-: no longer names the net of CR25.2, J9.2, Q26.2 (C_1), Q26.4 (C_2)
- net Valve13-: no longer names the net of CR29.2, J9.4, Q30.2 (C_1), Q30.4 (C_2)
- net Valve14-: no longer names the net of CR33.2, J9.6, Q34.2 (C_1), Q34.4 (C_2)
- net Valve15-: no longer names the net of CR36.2, J30.2, Q37.2 (C_1), Q37.4 (C_2)
- net Valve18-: no longer names the net of CR30.2, J37.4, Q31.2 (C_1), Q31.4 (C_2)
- net Valve2-: no longer names the net of CR23.2, J29.4, Q24.2 (C_1), Q24.4 (C_2)
- net Valve3-: no longer names the net of CR27.2, J29.6, Q28.2 (C_1), Q28.4 (C_2)
- net Valve4-: no longer names the net of CR31.2, J7.2, Q32.2 (C_1), Q32.4 (C_2)
- net Valve5-: no longer names the net of CR34.2, J31.2, Q35.2 (C_1), Q35.4 (C_2)
- net Valve6-: no longer names the net of CR20.2, J27.2, Q21.2 (C_1), Q21.4 (C_2)
- net Valve7-: no longer names the net of CR24.2, J31.4, Q25.2 (C_1), Q25.4 (C_2)
- net Valve8-: no longer names the net of CR28.2, J31.6, Q29.2 (C_1), Q29.4 (C_2)
- new net: R78.1, U15.27 (*SYNC), U20.91 (PB5)
Other:
- note added: "+12VB Voltage Plane is the regulated voltage from Vbat. +12VA is a seperate voltage plane used for powering all valves."
- note added: "AD7124-8 Pressure Measurments"
- note added: "KEY"
- note added: "Pressure Sensor Connection"
- note added: "Test Points"
- note removed: ".02 A (20mA max from pressure sensor) * 125 = 2.5 V (2.5 volt max reading from ad7124)"
- note removed: "Breakouts"
- note removed: "Heater"
- note removed: "PT"
- note removed: "TC"
- note removed: "UART Lines"
- note removed: "Valves"
- moved on the sheet: C145, C146, C147, C148, C149, C150, C151, C152, C153, C154, C155, C156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

Commit message: Circuit Diagram Done
Connections:
- net *SYNC is gone; now on an unnamed net: J33.5 (Pin_5)
- net ADC is gone; now on an unnamed net: J33.4 (Pin_4)
- net SPI1_MISO is gone; now on an unnamed net: J33.1 (Pin_1)
- net SPI1_MOSI is gone; now on an unnamed net: J33.2 (Pin_2)
- net SPI1_SCK is gone; now on an unnamed net: J33.3 (Pin_3)
- net SPI2_MISO is gone; now on an unnamed net: J12.1 (Pin_1)
- net SPI2_MOSI is gone; now on an unnamed net: J12.2 (Pin_2)
- net SPI2_SCK is gone; now on an unnamed net: J12.3 (Pin_3)
- net T1 is gone; now on an unnamed net: J39.5 (Pin_5)
- net T2 is gone; now on an unnamed net: J39.4 (Pin_4)
- net T3 is gone; now on an unnamed net: J39.3 (Pin_3)
- net T4 is gone; now on an unnamed net: J39.2 (Pin_2)
- net T5 is gone; now on an unnamed net: J39.1 (Pin_1)
- net UART_PPU_RX is gone; now on an unnamed net: J40.4
- net UART_PPU_TX is gone; now on an unnamed net: J40.3
- net +12VA: now also CR21.1
- net at U20.84 (PD3), U23.11 (SDO), U24.11 (SDO)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: no longer U27.11 (SDO)
- net at U20.85 (PD4), U23.12 (SDI), U24.12 (SDI)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: now also U27.11 (SDO)
- net I2C4_SCL: no longer names the net of J38.2, R27.2, U20.47 (PB10)
- net I2C4_SDA: no longer names the net of J38.1, R28.2, U20.48 (PB11)
- net PT: no longer names the net of J39.6 (Pin_6), U20.3 (PE4), U28.32 (*CS)
- net Valve10-: no longer names the net of CR35.2, J32.4, Q36.2 (C_1), Q36.4 (C_2)
- net Valve11-: no longer names the net of CR21.2, J32.6, Q22.2 (C_1), Q22.4 (C_2)
- net Valve9-: no longer names the net of CR32.2, J32.2, Q33.2 (C_1), Q33.4 (C_2)
Other:
- note added: "T1"
- note added: "T3"
- note added: "T4"
- note added: "T5"
- moved on the sheet: C100, C101, C102, C103, C104, C105, C106, C107, C108, C109, C110, C111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
