File: hw/Demo/led_solenoid_valve_pcb/led_solenoid_valve_pcb.kicad_sch (KiCad schematic)
At the start: 3 parts, among them J1 Conn_01x02

Commit message: LED SOLENOID PCB Reviewed: ERC + DRC Pass
Other:
- note added: "Solenoid LED Connector"
Changed lines of the file:
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@@
+		)
+	)
+	(text "Solenoid LED Connector\n"
+		(exclude_from_sim no)
+		(at 29.972 15.748 0)
+		(effects
+			(font
+				(size 1.27 1.27)
+			)
 		)
 	)
@@
 		)
 	)
-	(label "LED"
-		(at 19.05 16.51 0)
-		(effects
-			(font
-				(size 1.27 1.27)
-			)
-			(justify left bottom)
-		)
-	)
