File: hw/Breakout_board/monarch_breakout_board_rev2/monarch_breakout_board_rev2.kicad_sch (KiCad schematic)
At the start: 14 parts, among them U1 FDC2214RGHR, U2 INA226AQDGSRQ1

Commit message: ADXL355 Schematic Addition + I2C Problem within the chip
Parts:
- added C10, C12, C13, C8: 0.1uF, Capacitor_SMD:C_0603_1608Metric, symbol Device:C
- added C7, C9: 1uF, Capacitor_SMD:C_0603_1608Metric, symbol Device:C
- added R2, R3: 100k, symbol Device:R_US
- added R4: 0, symbol Device:R_US
- added U3: ADXL355BEZ, ADXL355:E_14_1-M, symbol ADXL355:ADXL355BEZ
- U1: renamed from U2; footprint DGS10_TEX -> INA226-Q1:DGS10_TEX
- renumbered U1 to U2
Connections:
- net +3V3: now also C10.1, C7.1, C8.1, C9.1, U3.11 (VSUPPLY), U3.5 (VDDIO)
- net GND: now also C10.2, C12.2, C13.2, C7.2, C8.2, C9.2, R2.2, R3.2, U3.4 (MISO/ASEL), U3.6 (VSSIO), U3.9 (VSSIO_2)
- net I2C4_SCL: now also R4.1
- net I2C4_SDA: now also U3.3 (MOSI/SDA)
- new net: C13.1, R3.1, U3.10 (V1P8NA)
- new net: R4.2, U3.1 (CSN/SCL)
- new net: C12.1, R2.1, U3.8 (V1P8DIG)
Other:
- sheet Connectors ports: added Cap0+, Cap0-, Cap1+, Cap1-, Cap2+, Cap2-, Cap3+, Cap3-, I2C4_SCL, I2C4_SDA; removed none
- note added: "I2C Addr: 0x1D"
- note added: "dilemma with the I2C bus problem"
- note added: "sets the addr to 0x1D"

Commit message: Charge probe resistor divided added
Parts:
- added R5, R6: ?, Resistor_SMD:R_0603_1608Metric_Pad0.98x0.95mm_HandSolder, symbol Device:R_US
Connections:
- net GND: now also U3.2 (SCLK/VSSIO), R5.1
- new net: R5.2, R6.1
- no-connect marks 2 -> 6
Other:
- note added: "Charge Probe Voltage Divider"
- note added: "I2C Mode Enable -> sets I2C mode"
- note added: "dilemma with the I2C bus problem (we could manipulate pin 2 with a gpio pin"
- note added: "need to check 1-4 pins on exmaple schematics"
- note added: "shunt voltage range INA226-Q1 measures +/- 81.92 mV"
- note removed: "dilemma with the I2C bus problem"
