File: hw/Breakout_boards/Accelerometer_Board/untitled.kicad_sch (KiCad schematic)
At the start: 14 parts, among them J3 2200980471, J4 2200980471

Commit message: Breakout Boards Measurements
Parts:
- removed TP5, TP6, TP7, TP8: TestPoint, TestPoint:TestPoint_Keystone_5000-5004_Miniature, symbol Connector:TestPoint
Other:
- note added: "will become 6 connector if switch to spi"
