File: hw/Breakout_boards/Plume_Measurment_Board/untitled.kicad_sch (KiCad schematic)
At the start: 14 parts, among them J3 2200980471, J4 2200980471

Commit message: Accelerometer Board Removed
Parts:
- removed H1, H2, H3, H4: MountingHole, MountingHole:MountingHole_2.2mm_M2_DIN965_Pad, symbol Mechanical:MountingHole
- removed J3, J4: 2200980471, Connector_Molex_Micro-Lock-Plus:Molex_Micro-Lock_2200980471_1x04_P1.25mm_Horizontal, symbol 5037630491:5037630491
- removed TP1, TP2, TP3, TP4, TP5, TP6, TP7, TP8: TestPoint, TestPoint:TestPoint_Keystone_5000-5004_Miniature, symbol Connector:TestPoint
Other:
- note removed: "Breakout Board Connection"
- note removed: "Mounting Holes"
- note removed: "PIB Connection"
