File: hw/Breakout_boards/Plume_Measurment_Board/Plume_Measurement_Board_REV2/Plume_Measurment_Board.kicad_sch (KiCad schematic)
At the start: 15 parts, among them J1 Conn_Coaxial, U1 AD7124-8BCPZ-RL

Commit message: Addedd Symbols Libraries
Connections:
- net PT renamed ESP
- net SPI2_MISO renamed SPI1_MISO
- net SPI2_MOSI renamed SPI1_MOSI
- net SPI2_SCK renamed SPI1_SCK
Changed lines of the file:
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@@
 		)
 	)
-	(hierarchical_label "SPI2_MISO"
+	(hierarchical_label "SPI1_MISO"
 		(shape output)
 		(at 121.92 121.92 0)
@@
 		)
 	)
-	(hierarchical_label "SPI2_MOSI"
+	(hierarchical_label "SPI1_MOSI"
 		(shape input)
 		(at 121.92 119.38 0)
@@
 		)
 	)
-	(hierarchical_label "PT"
+	(hierarchical_label "ESP"
 		(shape input)
 		(at 121.92 111.76 0)
@@
 		)
 	)
-	(hierarchical_label "SPI2_SCK"
+	(hierarchical_label "SPI1_SCK"
 		(shape bidirectional)
 		(at 121.92 116.84 0)
