File: hw/Breakout_boards/Capacitance_Measurement_Board/monarch_breakout_board_rev2/monarch_breakout_board_rev2.kicad_sch (KiCad schematic)
At the start: 13 parts, among them U2 FDC2214RGHR

Commit message: Breakout Boards Measurements
Changed lines of the file:
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@@
+		)
+	)
+	(label "board revision do we want to keep this differential pair setup?"
+		(at -54.61 45.72 0)
+		(effects
+			(font
+				(size 1.27 1.27)
+			)
+			(justify left bottom)
 		)
 	)
@@
 			(project "monarch_breakout_board_rev2"
 				(path "/7f71233a-1f17-423c-a2e8-36ba020ec1ce"
-					(page "3")
-				)
-			)
+					(page "2")
+				)
+			)

Commit message: New REV2 Breakout Board Schematic Done
Parts:
- added C10, C11, C12, C13, C14, C15, C16, C17, C18, C19, C20, C21, C22, C7, C8, C9: 18pF, Capacitor_SMD:C_0603_1608Metric, symbol Device:C
Connections:
- net Cap0+: now also C8.1, C9.1
- net Cap0-: now also C10.2, C7.2
- net Cap1+: now also C11.1, C13.1
- net Cap1-: now also C12.2, C14.2
- net Cap2+: now also C15.1, C17.1
- net Cap2-: now also C16.2, C18.2
- net Cap3+: now also C19.1, C21.1
- net Cap3-: now also C20.2, C22.2
- net GND: now also C10.1, C11.2, C12.1, C13.2, C14.1, C15.2, C16.1, C17.2, C18.1, C19.2, C20.1, C21.2, C22.1, C7.1, C8.2, C9.2
Other:
- moved on the sheet: C1, C5, C6, D1, L1, R1, U2

Commit message: Capacitance Board Schematic Done - Ran into issue with too big of BNC connectors
Parts:
- removed L1, L2, L3, L4: 18uH, Inductor_SMD:L_0805_2012Metric, symbol Device:L
- added L1, L2, L3, L4: 18uH, Inductor_Bourns:INDM3225X240N, symbol Device:L_Iron
- renumbered C16 to C10, C19 to C11, C20 to C12, C9 to C15, C10 to C16, C21 to C19, C22 to C20, C5 to C21, C6 to C22, C11 to C5, C12 to C6, C8 to C7, C7 to C8, C15 to C9, U2 to U1
Connections:
- net Cap0+: now also L1.1
- net Cap0-: now also L1.2
- net Cap1+: now also L2.1
- net Cap1-: now also L2.2
- net Cap2+: now also L3.1
- net Cap2-: now also L3.2
- net Cap3+: now also L4.1
- net Cap3-: now also L4.2
Other:
- moved on the sheet: C2

Commit message: Close Valve Cmds implementation + AD7124 + port over correct drivers
Other:
- title: Breakout Board -> Capacitance Measurement Board
Changed lines of the file:
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@@
 	(paper "A4")
 	(title_block
-		(title "Breakout Board")
+		(title "Capacitance Measurement Board")
 		(date "2026-08-04")
 		(rev "REV_2")
