File: hw/Breakout_boards/Capacitance_Measurement_Board/monarch_breakout_board_rev2/monarch_breakout_board_rev2.kicad_pcb (KiCad board)
At the start: 2 copper layers, 24.6 x 27.1 mm, 42 parts, among them J1 Conn_01x02, J2 Conn_01x02, J3 Conn_01x02, J4 Conn_01x02, J9 2200980471, U1 FDC2214RGHR

Commit message: 3-D Models Added
Parts:
- moved H1 0.31 mm to (109.7, 41.7)
- moved H2 0.30 mm to (109.7, 63.7)
Routing:
- net GND: track 54.6 -> 64.1 mm
Other:
- board size 24.6 x 27.1 mm -> 24.4 x 26.9 mm
Changed lines of the file:
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@@
 		)
 		(embedded_fonts no)
-		(model "CM322522-180KL.stp"
+		(model "${KIPRJMOD}/CM322522-180KL/3D/CM322522-180KL.stp"
 			(offset
 				(xyz 0 -0.1500000037 0.01999999925)
@@
 		)
 		(embedded_fonts no)
-		(model "CM322522-180KL.stp"
+		(model "${KIPRJMOD}/CM322522-180KL/3D/CM322522-180KL.stp"
 			(offset
 				(xyz 0 -0.1500000037 0.01999999925)
@@
 		)
 		(embedded_fonts no)
+		(model "${KIPRJMOD}/FDC2214/RGH0016A.stp"
+			(offset
+				(xyz 0 0 0)
+			)
+			(scale
+				(xyz 1 1 1)
+			)
+			(rotate
+				(xyz 0 0 0)
+			)
+		)
 	)
 	(footprint "Capacitor_SMD:C_0603_1608Metric"
@@
 	(footprint "MountingHole:MountingHole_2.2mm_M2_DIN965_Pad"
 		(layer "F.Cu")
-		(at 128.999967 41.604098 90)
+		(at 129.032 41.604098 90)
 		(descr "Mounting Hole 2.2mm, M2, generated by kicad-footprint-generator mountinghole.py")
 		(tags "mountinghole M2 DIN965")
@@
 		)
 		(embedded_fonts no)
-		(model "CM322522-180KL.stp"
+		(model "${KIPRJMOD}/CM322522-180KL/3D/CM322522-180KL.stp"
 			(offset
 				(xyz 0 -0.1500000037 0.01999999925)
@@
 	(footprint "MountingHole:MountingHole_2.2mm_M2_DIN965_Pad"
 		(layer "F.Cu")
-		(at 109.425 41.725 90)
+		(at 109.728 41.656 90)
 		(descr "Mounting Hole 2.2mm, M2, generated by kicad-footprint-generator mountinghole.py")
 		(tags "mountinghole M2 DIN965")
@@
 	(footprint "MountingHole:MountingHole_2.2mm_M2_DIN965_Pad"
 		(layer "F.Cu")
-		(at 129.012777 63.616341 90)
+		(at 129.032 63.616341 90)
 		(descr "Mounting Hole 2.2mm, M2, generated by kicad-footprint-generator mountinghole.py")
 		(tags "mountinghole M2 DIN965")
@@
 		)
 		(embedded_fonts no)
+		(model "${KIPRJMOD}/Connector_Molex_Micro-Lock-Plus/Connector_Molex_Micro-Lock-Plus.pretty/3D-Models/2200980471.stp"
+			(offset
+				(xyz 0 0 0)
+			)
+			(scale
+				(xyz 1 1 1)
+			)
+			(rotate
+				(xyz -90 -0 -0)
+			)
+		)
 	)
 	(footprint "TestPoint:TestPoint_Keystone_5000-5004_Miniature"
@@
 	(footprint "MountingHole:MountingHole_2.2mm_M2_DIN965_Pad"
 		(layer "F.Cu")
-		(at 109.425 63.725 90)
+		(at 109.728 63.725 90)
 		(descr "Mounting Hole 2.2mm, M2, generated by kicad-footprint-generator mountinghole.py")
 		(tags "mountinghole M2 DIN965")
@@
 		)
 		(embedded_fonts no)
-		(model "CM322522-180KL.stp"
+		(model "${KIPRJMOD}/CM322522-180KL/3D/CM322522-180KL.stp"
 			(offset
 				(xyz 0 -0.1500000037 0.01999999925)
@@
 	)
 	(gr_line
-		(start 106.925 41.725)
-		(end 106.925 63.75)
+		(start 107.188 41.656)
+		(end 107.188 63.5)
 		(stroke
 			(width 0.05)
@@
 	)
 	(gr_arc
-		(start 106.925 41.725)
-		(mid 107.657233 39.957233)
-		(end 109.425 39.225)
+		(start 107.188 41.656)
+		(mid 107.931949 39.859949)
+		(end 109.728 39.116)
 		(stroke
 			(width 0.05)
@@
 	)
 	(gr_arc
-		(start 109.425 66.225)
-		(mid 107.657233 65.492767)
-		(end 106.925 63.725)
+		(start 109.728 66.04)
+		(mid 107.931949 65.296051)
+		(end 107.188 63.5)
 		(stroke
 			(width 0.05)
@@
 	)
 	(gr_line
-		(start 109.425 66.225)
-		(end 129.047489 66.109144)
+		(start 109.728 66.04)
+		(end 129.032 66.04)
 		(stroke
 			(width 0.05)
@@
 	)
 	(gr_line
-		(start 129 39.104065)
-		(end 109.424885 39.225)
+		(start 129.032 39.116)
+		(end 109.728 39.116)
 		(stroke
 			(width 0.05)
@@
 	)
 	(gr_arc
-		(start 129 39.104065)
-		(mid 130.767767 39.836298)
-		(end 131.5 41.604065)
+		(start 129.032 39.116)
+		(mid 130.828051 39.859949)
+		(end 131.572 41.656)
 		(stroke
 			(width 0.05)
@@
 	)
 	(gr_arc
-		(start 131.505577 63.584141)
-		(mid 130.786969 65.367741)
-		(end 129.01281 66.109349)
+		(start 131.572 63.5)
+		(mid 130.828051 65.296051)
+		(end 129.032 66.04)
 		(stroke
 			(width 0.05)
@@
 	)
 	(gr_line
-		(start 131.505577 63.584221)
-		(end 131.5 41.604065)
+		(start 131.572 63.5)
+		(end 131.572 41.656)
 		(stroke
 			(width 0.05)
@@
 	)
 	(segment
+		(start 114.799999 54.599999)
+		(end 113.500001 54.599999)
+		(width 0.2)
+		(layer "F.Cu")
+		(net "GND")
+	)
+	(segment
 		(start 108.4 56.325)
 		(end 108.8 55.925)
@@
 	)
 	(segment
+		(start 118 58.486525)
+		(end 118.00048 58.487005)
+		(width 0.2)
+		(layer "F.Cu")
+		(net "GND")
+	)
+	(segment
+		(start 118 56.95)
+		(end 118 58.486525)
+		(width 0.2)
+		(layer "F.Cu")
+		(net "GND")
+	)
+	(segment
 		(start 126.5 47.025)
 		(end 126.5 46.4)
@@
 	)
 	(segment
+		(start 117.449999 56.399999)
+		(end 118 56.95)
+		(width 0.2)
+		(layer "F.Cu")
+		(net "GND")
+	)
+	(segment
 		(start 115.949997 54.599999)
 		(end 116.699998 53.849998)
@@
 	)
 	(segment
+		(start 118.00048 59.12452)
+		(end 116.3104 60.8146)
+		(width 0.2)
+		(layer "F.Cu")
+		(net "GND")
+	)
+	(segment
+		(start 116.3104 60.8146)
+		(end 116.3104 61.101201)
+		(width 0.2)
+		(layer "F.Cu")
+		(net "GND")
+	)
+	(segment
+		(start 117.449999 55.75)
+		(end 117.449999 56.399999)
+		(width 0.2)
+		(layer "F.Cu")
+		(net "GND")
+	)
+	(segment
+		(start 118.00048 58.487005)
+		(end 118.00048 59.12452)
+		(width 0.2)
+		(layer "F.Cu")
+		(net "GND")
+	)
+	(segment
 		(start 114.799999 54.599999)
 		(end 115.949997 54.599999)
 		(width 0.2)
 		(layer "F.Cu")
+		(net "GND")
+	)
+	(segment
+		(start 113.500001 54.599999)
+		(end 112.15 55.95)
+		(width 0.2)
+		(layer "F.Cu")

Commit message: DRC PASS
Parts:
- moved C5 0.60 mm to (124.0, 52.4)
- moved C14 0.50 mm to (121.0, 52.4)
Routing:
- net GND: track 64.1 -> 64.0 mm, vias 5 -> 3
Other:
- board text added: "Breakout Board - Capacitance"
- board text added: "Rev2 - 08/06/2026"
- board text removed: "Breakout Board"
- board text removed: "Rev2 - 08//2026"
