File: hw/Breakout_boards/Plume_Measurment_Board/Plume_Measurement_Board_REV1/E-Spray_Plume_Measurement_1.kicad_sch (KiCad schematic)
At the start: 35 parts, among them J5 Conn_Coaxial, U2 LMP7721MA/NOPB, U3 LMP2022MA/NOPB, U4 AD8475ARMZ, U5 AD8475ARMZ, U7 AD7176-2BRUZ

Commit message: Mirrored Layout Finish
Changed lines of the file:
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@@
-	(wire
-		(pts
-			(xy 0.0762 0.8096) (xy 5.1562 0.8096)
-		)
-		(stroke
-			(width 0)
-			(type default)
-		)
-	)
 	(wire
 		(pts
@@
 			(width 0)
 			(type default)
-		)
-	)
-	(hierarchical_label "VSS"
-		(shape input)
-		(at 5.1562 0.8096 0)
-		(effects
-			(font
-				(size 1.27 1.27)
-			)
-			(justify left)
 		)
 	)
@@
 		)
 	)
+	(rule_area
+		(exclude_from_sim no)
+		(in_bom yes)
+		(on_board yes)
+		(dnp no)
+		(polyline
+			(pts
+				(xy 11.43 11.43) (xy 11.43 199.39) (xy 285.75 199.39) (xy 287.02 198.12) (xy 287.02 10.16) (xy 12.7 10.16)
+			)
+			(stroke
+				(width 0)
+				(type dash)
+			)
+			(fill
+				(type none)
+			)
+		)
+	)
