File: hw/Breakout_boards/Plume_Measurment_Board/Plume_Measurement_Board_REV1/untitled.kicad_sch (KiCad schematic)
At the start: 0 parts

Commit message: Voltage Regulator Library Import + Connector Additions
Parts:
- added J2, J4: Conn_01x04, Connector_Molex_Micro-Lock-Plus:Molex_Micro-Lock_2200980471_1x04_P1.25mm_Horizontal, symbol Connector_Generic:Conn_01x04
Connections:
- new net +VBAT: J2.1 (Pin_1)
- new net 3V3: J2.3 (Pin_3)
- new net GND: J2.2 (Pin_2), J2.4 (Pin_4)
- new net PM_CS: J4.4 (Pin_4)
- new net SPI1_CLK: J4.3 (Pin_3)
- new net SPI1_MISO: J4.2 (Pin_2)
- new net SPI1_MOSI: J4.1 (Pin_1)
Other:
- note added: "Communication Protocol Connector"
- note added: "Power Connector"

Commit message: Orgnanization Between Pages
Parts:
- added J3: Conn_Coaxial, symbol Connector:Conn_Coaxial
Connections:
- net GND: now also J3.2 (Ext)
- new net Plume: J3.1 (In)
Other:
- note added: "E-spray Probe Connector"
Changed lines of the file:
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@@
 		)
 	)
-	(text "Communication Protocol Connector"
-		(exclude_from_sim no)
-		(at 85.598 16.51 0)
+	(rectangle
+		(start 157.48 12.7)
+		(end 228.6 63.5)
+		(stroke
+			(width 0)
+			(type dash)
+		)
+		(fill
+			(type none)
+		)
+	)
+	(text "E-spray Probe Connector\n"
+		(exclude_from_sim no)
+		(at 158.242 16.764 0)
 		(effects
 			(font
@@
 		)
 	)
-	(text "Power Connector\n"
-		(exclude_from_sim no)
-		(at 13.208 16.51 0)
+	(text "Communication Protocol Connector"
+		(exclude_from_sim no)
+		(at 85.598 16.51 0)
 		(effects
 			(font
@@
 		)
 	)
+	(text "Power Connector\n"
+		(exclude_from_sim no)
+		(at 13.208 16.51 0)
+		(effects
+			(font
+				(size 2 2)
+				(thickness 0.4)
+				(bold yes)
+			)
+			(justify left bottom)
+		)
+	)
 	(wire
 		(pts
@@
 		(shape input)
 		(at 116.84 34.29 180)
+		(effects
+			(font
+				(size 1.27 1.27)
+			)
+			(justify right)
+		)
+	)
+	(hierarchical_label "Plume"
+		(shape input)
+		(at 187.96 35.56 180)
 		(effects
 			(font
@@
 	)
 	(symbol
+		(lib_id "Connector:Conn_Coaxial")
+		(at 193.04 35.56 0)
+		(unit 1)
+		(body_style 1)
+		(exclude_from_sim no)
+		(in_bom yes)
+		(on_board yes)
+		(in_pos_files yes)
+		(dnp no)
+		(fields_autoplaced yes)
+		(property "Reference" "J3"
+			(at 196.85 34.5831 0)
+			(show_name no)
+			(do_not_autoplace no)
+			(effects
+				(font
+					(size 1.27 1.27)
+				)
+				(justify left)
+			)
+		)
+		(property "Value" "Conn_Coaxial"
+			(at 196.85 37.1231 0)
+			(show_name no)
+			(do_not_autoplace no)
+			(effects
+				(font
+					(size 1.27 1.27)
+				)
+				(justify left)
+			)
+		)
+		(property "Footprint" ""
+			(at 193.04 35.56 0)
+			(hide yes)
+			(show_name no)
+			(do_not_autoplace no)
+			(effects
+				(font
+					(size 1.27 1.27)
+				)
+			)
+		)
+		(property "Datasheet" ""
+			(at 193.04 35.56 0)
+			(hide yes)
+			(show_name no)
+			(do_not_autoplace no)
+			(effects
+				(font
+					(size 1.27 1.27)
+				)
+			)
+		)
+		(property "Description" "coaxial connector (BNC, SMA, SMB, SMC, Cinch/RCA, LEMO, ...)"
+			(at 193.04 35.56 0)
+			(hide yes)
+			(show_name no)
+			(do_not_autoplace no)
+			(effects
+				(font
+					(size 1.27 1.27)
+				)
+			)
+		)
+		(pin "2"
+		)
+		(pin "1"
+		)
+		(instances
+			(project "Plume_Measurment_Board"
+				(path "/2e1d3673-27b9-4604-80fb-036cec98a912/4097d861-b189-461e-b768-3d03272bff16"
+					(reference "J3")
+					(unit 1)
+				)
+			)
+		)
+	)
+	(symbol
 		(lib_id "Connector_Generic:Conn_01x04")
 		(at 121.92 34.29 0)
@@
 					(unit 1)
 				)
+			)
+		)
+	)
+	(symbol
+		(lib_id "power:GND")
+		(at 193.04 40.64 0)
+		(unit 1)
+		(body_style 1)
+		(exclude_from_sim no)
+		(in_bom yes)
+		(on_board yes)
+		(in_pos_files yes)
+		(dnp no)
+		(fields_autoplaced yes)
+		(property "Reference" "#PWR03"
+			(at 193.04 46.99 0)
+			(hide yes)
+			(show_name no)
+			(do_not_autoplace no)
+			(effects
+				(font
+					(size 1.27 1.27)
+				)
+			)
+		)
+		(property "Value" "GND"
+			(at 193.04 45.72 0)
+			(show_name no)
+			(do_not_autoplace no)
+			(effects
+				(font
+					(size 1.27 1.27)
+				)
+			)
+		)
+		(property "Footprint" ""
+			(at 193.04 40.64 0)
+			(hide yes)
+			(show_name no)
+			(do_not_autoplace no)
+			(effects
+				(font
+					(size 1.27 1.27)
+				)
+			)
+		)
+		(property "Datasheet" ""
+			(at 193.04 40.64 0)
+			(hide yes)
+			(show_name no)
+			(do_not_autoplace no)
+			(effects
+				(font
+					(size 1.27 1.27)
+				)
+			)
+		)
+		(property "Description" "Power symbol creates a global label with name \"GND\" , ground"
+			(at 193.04 40.64 0)
+			(hide yes)
+			(show_name no)
+			(do_not_autoplace no)
+			(effects
+				(font
+					(size 1.27 1.27)
+				)
+			)
+		)
+		(pin "1"
+		)
+		(instances
+			(project "Plume_Measurment_Board"
+				(path "/2e1d3673-27b9-4604-80fb-036cec98a912/4097d861-b189-461e-b768-3d03272bff16"
+					(reference "#PWR03")
+					(unit 1)
+				)

Commit message: Connector Fixes
Connections:
- net 3V3 renamed +3V3
Other:
- company: (none) -> Electric Propulsion Lab
- title: (none) -> Plume Measurement Board
Changed lines of the file:
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@@
 	(generator_version "10.0")
 	(paper "A4")
+	(title_block
+		(title "Plume Measurement Board")
+		(date "2026-08-06")
+		(rev "REV1")
+		(company "Electric Propulsion Lab")
+		(comment 4 "Kacper Paraniuk")
+	)
 	(rectangle
 		(start 85.09 12.7)
@@
 	(wire
 		(pts
-			(xy 34.29 35.56) (xy 34.29 34.29)
+			(xy 33.02 35.56) (xy 33.02 34.29)
 		)
 		(stroke
@@
 	(wire
 		(pts
-			(xy 34.29 34.29) (xy 46.99 34.29)
+			(xy 36.83 36.83) (xy 36.83 30.48)
+		)
+		(stroke
+			(width 0)
+			(type default)
+		)
+	)
+	(wire
+		(pts
+			(xy 33.02 34.29) (xy 46.99 34.29)
 		)
 		(stroke
@@
 		)
 	)
+	(wire
+		(pts
+			(xy 46.99 36.83) (xy 36.83 36.83)
+		)
+		(stroke
+			(width 0)
+			(type default)
+		)
+	)
 	(hierarchical_label "PM_CS"
 		(shape output)
 		(at 116.84 39.37 180)
-		(effects
-			(font
-				(size 1.27 1.27)
-			)
-			(justify right)
-		)
-	)
-	(hierarchical_label "3V3"
-		(shape input)
-		(at 46.99 36.83 180)
 		(effects
 			(font
@@
 	(symbol
 		(lib_id "power:GND")
-		(at 34.29 35.56 0)
+		(at 33.02 35.56 0)
 		(unit 1)
 		(body_style 1)
@@
 		(fields_autoplaced yes)
 		(property "Reference" "#PWR01"
-			(at 34.29 41.91 0)
+			(at 33.02 41.91 0)
 			(hide yes)
 			(show_name no)
@@
 		)
 		(property "Value" "GND"
-			(at 34.29 40.64 0)
+			(at 33.02 40.64 0)
 			(show_name no)
 			(do_not_autoplace no)
@@
 		)
 		(property "Footprint" ""
-			(at 34.29 35.56 0)
+			(at 33.02 35.56 0)
 			(hide yes)
 			(show_name no)
@@
 		)
 		(property "Datasheet" ""
-			(at 34.29 35.56 0)
+			(at 33.02 35.56 0)
 			(hide yes)
 			(show_name no)
@@
 		)
 		(property "Description" "Power symbol creates a global label with name \"GND\" , ground"
-			(at 34.29 35.56 0)
+			(at 33.02 35.56 0)
 			(hide yes)
 			(show_name no)
@@
 					(unit 1)
 				)
+			)
+		)
+	)
+	(symbol
+		(lib_id "power:+3V3")
+		(at 36.83 30.48 0)
+		(unit 1)
+		(body_style 1)
+		(exclude_from_sim no)
+		(in_bom yes)
+		(on_board yes)
+		(in_pos_files yes)
+		(dnp no)
+		(property "Reference" "#PWR0246"
+			(at 36.83 34.29 0)
+			(hide yes)
+			(show_name no)
+			(do_not_autoplace no)
+			(effects
+				(font
+					(size 1.27 1.27)
+				)
+			)
+		)
+		(property "Value" "+3V3"
+			(at 36.83 26.67 0)
+			(show_name no)
+			(do_not_autoplace no)
+			(effects
+				(font
+					(size 1.27 1.27)
+				)
+			)
+		)
+		(property "Footprint" ""
+			(at 36.83 30.48 0)
+			(hide yes)
+			(show_name no)
+			(do_not_autoplace no)
+			(effects
+				(font
+					(size 1.27 1.27)
+				)
+			)
+		)
+		(property "Datasheet" ""
+			(at 36.83 30.48 0)
+			(hide yes)
+			(show_name no)
+			(do_not_autoplace no)
+			(effects
+				(font
+					(size 1.27 1.27)
+				)
+			)
+		)
+		(property "Description" "Power symbol creates a global label with name \"+3V3\""
+			(at 36.83 30.48 0)
+			(hide yes)
+			(show_name no)
+			(do_not_autoplace no)
+			(effects
+				(font
+					(size 1.27 1.27)
+				)
+			)
+		)
+		(pin "1"
+		)
+		(instances
+			(project "Plume_Measurment_Board"
+				(path "/2e1d3673-27b9-4604-80fb-036cec98a912/4097d861-b189-461e-b768-3d03272bff16"
+					(reference "#PWR0246")
+					(unit 1)
+				)

Commit message: Entire RF pipeline
Parts:
- J3: footprint (none) -> Connector_Coaxial:SMA_Molex_73251-2120_EdgeMount_Horizontal
Connections:
- net GND: no longer J3.2 (Ext)
- new net +2.5V: J3.2 (Ext)
Changed lines of the file:
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@@
+	(wire
+		(pts
+			(xy 193.04 40.64) (xy 193.04 46.99)
+		)
+		(stroke
+			(width 0)
+			(type default)
+		)
+	)
 	(wire
 		(pts
@@
 		(shape input)
 		(at 187.96 35.56 180)
+		(effects
+			(font
+				(size 1.27 1.27)
+			)
+			(justify right)
+		)
+	)
+	(hierarchical_label "+2.5V"
+		(shape input)
+		(at 193.04 46.99 180)
 		(effects
 			(font
@@
 			)
 		)
-		(property "Footprint" ""
+		(property "Footprint" "Connector_Coaxial:SMA_Molex_73251-2120_EdgeMount_Horizontal"
 			(at 193.04 35.56 0)
 			(hide yes)
@@
 					(unit 1)
 				)
-			)
-		)
-	)
-	(symbol
-		(lib_id "power:GND")
-		(at 193.04 40.64 0)
-		(unit 1)
-		(body_style 1)
-		(exclude_from_sim no)
-		(in_bom yes)
-		(on_board yes)
-		(in_pos_files yes)
-		(dnp no)
-		(fields_autoplaced yes)
-		(property "Reference" "#PWR03"
-			(at 193.04 46.99 0)
-			(hide yes)
-			(show_name no)
-			(do_not_autoplace no)
-			(effects
-				(font
-					(size 1.27 1.27)
-				)
-			)
-		)
-		(property "Value" "GND"
-			(at 193.04 45.72 0)
-			(show_name no)
-			(do_not_autoplace no)
-			(effects
-				(font
-					(size 1.27 1.27)
-				)
-			)
-		)
-		(property "Footprint" ""
-			(at 193.04 40.64 0)
-			(hide yes)
-			(show_name no)
-			(do_not_autoplace no)
-			(effects
-				(font
-					(size 1.27 1.27)
-				)
-			)
-		)
-		(property "Datasheet" ""
-			(at 193.04 40.64 0)
-			(hide yes)
-			(show_name no)
-			(do_not_autoplace no)
-			(effects
-				(font
-					(size 1.27 1.27)
-				)
-			)
-		)
-		(property "Description" "Power symbol creates a global label with name \"GND\" , ground"
-			(at 193.04 40.64 0)
-			(hide yes)
-			(show_name no)
-			(do_not_autoplace no)
-			(effects
-				(font
-					(size 1.27 1.27)
-				)
-			)
-		)
-		(pin "1"
-		)
-		(instances
-			(project "Plume_Measurment_Board"
-				(path "/2e1d3673-27b9-4604-80fb-036cec98a912/4097d861-b189-461e-b768-3d03272bff16"
-					(reference "#PWR03")
-					(unit 1)
-				)

Commit message: New Schematic w/ Addition of two E-spray Amplification Signals
Parts:
- removed J3: Conn_Coaxial, Connector_Coaxial:SMA_Molex_73251-2120_EdgeMount_Horizontal, symbol Connector:Conn_Coaxial
Connections:
- net GND: no longer J2.4 (Pin_4)
- net PM_CS renamed PM_CS_2
- new net PM_CS_1: J2.4 (Pin_4)
Other:
- note removed: "E-spray Probe Connector"
Changed lines of the file:
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@@
-		)
-	)
-	(rectangle
-		(start 157.48 12.7)
-		(end 228.6 63.5)
-		(stroke
-			(width 0)
-			(type dash)
-		)
-		(fill
-			(type none)
-		)
-	)
-	(text "E-spray Probe Connector\n"
-		(exclude_from_sim no)
-		(at 158.242 16.764 0)
-		(effects
-			(font
-				(size 2 2)
-				(thickness 0.4)
-				(bold yes)
-			)
-			(justify left bottom)
 		)
 	)
@@
 			)
 			(justify left bottom)
-		)
-	)
-	(wire
-		(pts
-			(xy 193.04 40.64) (xy 193.04 46.99)
-		)
-		(stroke
-			(width 0)
-			(type default)
 		)
 	)
@@
 	(wire
 		(pts
-			(xy 46.99 39.37) (xy 39.37 39.37)
-		)
-		(stroke
-			(width 0)
-			(type default)
-		)
-	)
-	(wire
-		(pts
-			(xy 39.37 39.37) (xy 39.37 40.64)
-		)
-		(stroke
-			(width 0)
-			(type default)
-		)
-	)
-	(wire
-		(pts
 			(xy 46.99 36.83) (xy 36.83 36.83)
 		)
@@
 		)
 	)
-	(hierarchical_label "PM_CS"
+	(hierarchical_label "PM_CS_2"
 		(shape output)
 		(at 116.84 39.37 180)
@@
 		)
 	)
-	(hierarchical_label "Plume"
-		(shape input)
-		(at 187.96 35.56 180)
-		(effects
-			(font
-				(size 1.27 1.27)
-			)
-			(justify right)
-		)
-	)
-	(hierarchical_label "+2.5V"
-		(shape input)
-		(at 193.04 46.99 180)
+	(hierarchical_label "PM_CS_1"
+		(shape output)
+		(at 46.99 39.37 180)
 		(effects
 			(font
@@
 			)
 			(justify right)
-		)
-	)
-	(symbol
-		(lib_id "power:GND")
-		(at 39.37 40.64 0)
-		(unit 1)
-		(body_style 1)
-		(exclude_from_sim no)
-		(in_bom yes)
-		(on_board yes)
-		(in_pos_files yes)
-		(dnp no)
-		(fields_autoplaced yes)
-		(property "Reference" "#PWR02"
-			(at 39.37 46.99 0)
-			(hide yes)
-			(show_name no)
-			(do_not_autoplace no)
-			(effects
-				(font
-					(size 1.27 1.27)
-				)
-			)
-		)
-		(property "Value" "GND"
-			(at 39.37 45.72 0)
-			(show_name no)
-			(do_not_autoplace no)
-			(effects
-				(font
-					(size 1.27 1.27)
-				)
-			)
-		)
-		(property "Footprint" ""
-			(at 39.37 40.64 0)
-			(hide yes)
-			(show_name no)
-			(do_not_autoplace no)
-			(effects
-				(font
-					(size 1.27 1.27)
-				)
-			)
-		)
-		(property "Datasheet" ""
-			(at 39.37 40.64 0)
-			(hide yes)
-			(show_name no)
-			(do_not_autoplace no)
-			(effects
-				(font
-					(size 1.27 1.27)
-				)
-			)
-		)
-		(property "Description" "Power symbol creates a global label with name \"GND\" , ground"
-			(at 39.37 40.64 0)
-			(hide yes)
-			(show_name no)
-			(do_not_autoplace no)
-			(effects
-				(font
-					(size 1.27 1.27)
-				)
-			)
-		)
-		(pin "1"
-		)
-		(instances
-			(project "Plume_Measurment_Board"
-				(path "/2e1d3673-27b9-4604-80fb-036cec98a912/4097d861-b189-461e-b768-3d03272bff16"
-					(reference "#PWR02")
-					(unit 1)
-				)
-			)
 		)
 	)
@@
 					(unit 1)
 				)
-			)
-		)
-	)
-	(symbol
-		(lib_id "Connector:Conn_Coaxial")
-		(at 193.04 35.56 0)
-		(unit 1)
-		(body_style 1)
-		(exclude_from_sim no)
-		(in_bom yes)
-		(on_board yes)
-		(in_pos_files yes)
-		(dnp no)
-		(fields_autoplaced yes)
-		(property "Reference" "J3"
-			(at 196.85 34.5831 0)
-			(show_name no)
-			(do_not_autoplace no)
-			(effects
-				(font
-					(size 1.27 1.27)
-				)
-				(justify left)
-			)
-		)
-		(property "Value" "Conn_Coaxial"
-			(at 196.85 37.1231 0)
-			(show_name no)
-			(do_not_autoplace no)
-			(effects
-				(font
-					(size 1.27 1.27)
-				)
-				(justify left)
-			)
-		)
-		(property "Footprint" "Connector_Coaxial:SMA_Molex_73251-2120_EdgeMount_Horizontal"
-			(at 193.04 35.56 0)
-			(hide yes)
-			(show_name no)
-			(do_not_autoplace no)
-			(effects
-				(font
-					(size 1.27 1.27)
-				)
-			)
-		)
-		(property "Datasheet" ""
-			(at 193.04 35.56 0)
-			(hide yes)
-			(show_name no)
-			(do_not_autoplace no)
-			(effects
-				(font
-					(size 1.27 1.27)
-				)
-			)
-		)
-		(property "Description" "coaxial connector (BNC, SMA, SMB, SMC, Cinch/RCA, LEMO, ...)"
-			(at 193.04 35.56 0)
-			(hide yes)
-			(show_name no)
-			(do_not_autoplace no)
-			(effects
-				(font
-					(size 1.27 1.27)
-				)
-			)
-		)
-		(pin "2"
-		)
-		(pin "1"
-		)
-		(instances
-			(project "Plume_Measurment_Board"
-				(path "/2e1d3673-27b9-4604-80fb-036cec98a912/4097d861-b189-461e-b768-3d03272bff16"
-					(reference "J3")
-					(unit 1)
-				)

Commit message: Mech Drawing in User.Drawings + Progress Routing 5V regulator
Parts:
- added H1, H2, H3, H4: MountingHole, symbol Mechanical:MountingHole
Connections:
- net +VBAT: now also J2.4 (Pin_4); no longer J2.1 (Pin_1)
- net PM_CS_1: now also J4.4 (Pin_4); no longer J2.4 (Pin_4)
- net PM_CS_2: now also J2.1 (Pin_1); no longer J4.4 (Pin_4)
- net SPI1_MISO: now also J4.1 (Pin_1); no longer J4.2 (Pin_2)
- net SPI1_MOSI: now also J4.2 (Pin_2); no longer J4.1 (Pin_1)
Other:
- note added: "Mounting Holes"

Commit message: Edge Cuts Playing Around
Parts:
- H1, H2, H3, H4: footprint (none) -> MountingHole:MountingHole_3.5mm
Changed lines of the file:
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@@
 			)
 		)
-		(property "Footprint" ""
+		(property "Footprint" "MountingHole:MountingHole_3.5mm"
 			(at 199.39 43.18 0)
 			(hide yes)
@@
 			)
 		)
-		(property "Footprint" ""
+		(property "Footprint" "MountingHole:MountingHole_3.5mm"
 			(at 199.39 31.75 0)
 			(hide yes)
@@
 			)
 		)
-		(property "Footprint" ""
+		(property "Footprint" "MountingHole:MountingHole_3.5mm"
 			(at 179.07 31.75 0)
 			(hide yes)
@@
 			)
 		)
-		(property "Footprint" ""
+		(property "Footprint" "MountingHole:MountingHole_3.5mm"
 			(at 179.07 43.18 0)
 			(hide yes)

Commit message: Very interesting shape of board
Parts:
- removed H1, H2, H3, H4: MountingHole, MountingHole:MountingHole_3.5mm, symbol Mechanical:MountingHole
Other:
- note removed: "Mounting Holes"
