File: hw/Breakout_boards/Plume_Measurment_Board/Plume_Measurement_Board_REV1/untitled.kicad_sch (KiCad schematic)
At the start: 2 parts, among them J2 Conn_01x04, J4 Conn_01x04

Commit message: Hardware Debug Software Changes + New Mounting Holes for the Plume Measurement Board
Parts:
- added H1, H2, H3, H4: MountingHole, MountingHole:MountingHole_2.5mm, symbol Mechanical:MountingHole
Other:
- note added: "Mounting Holes"
